File: hardware/cpu/cpu.kicad_pcb (KiCad board)
At the start: 4 copper layers, 172.7 x 116.8 mm, 61 parts, among them J1 Conn_02x20_Odd_Even, J2 Conn_01x06, J3 Conn_01x06, J4 Conn_02x05_Odd_Even, J5 Conn_01x02, J6 Conn_02x20_Odd_Even, SW1 SW_Push, U1 74AS74, U10 74LS157, U11 Z80-DART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

Commit message: working on CPU
Parts:
- removed the REF** at (110.5, 138.4)
- removed the REF** at (110.5, 29.2)
- removed the REF** at (29.2, 29.2)
- added JP1: JPR3, Connector_PinHeader_2.54mm:PinHeader_1x03_P2.54mm_Vertical, F.Cu at (132.1, 82.5)
- added REF**: MountingHole_2.7mm_Pad, MountingHole:MountingHole_2.7mm_Pad, F.Cu at (28.6, 28.6)
- added REF**: lcd, lcd_mount:lcd, F.Cu at (39.4, 25.4)
- added U18: 74AS74, Package_DIP:DIP-14_W7.62mm_LongPads, F.Cu at (107.3, 100.3)
- C1: footprint Capacitor_SMD:C_0805_2012Metric -> Capacitor_THT:CP_Radial_D5.0mm_P2.50mm
- REF** (x3): value MountingHole_3.2mm_M3_Pad -> MountingHole_2.7mm_Pad; footprint MountingHole:MountingHole_3.2mm_M3_Pad -> MountingHole:MountingHole_2.7mm_Pad
- SW1: footprint Button_Switch_THT:SW_PUSH_6mm -> Connector_PinHeader_2.54mm:PinHeader_1x02_P2.54mm_Vertical
- X1: value 8.0000MHz -> 7.3728MHz; footprint Package_DIP:DIP-14_W7.62mm_Socket_LongPads -> Oscillator:Oscillator_DIP-8
- moved SW1 201.5 mm to (64.1, 127.6), turned to 90 degrees
- moved J2 167.3 mm to (87.0, 27.9), turned to 90 degrees
- moved J3 155.4 mm to (113.0, 27.9), turned to 90 degrees
- moved D2 116.9 mm to (128.3, 128.3)
- moved C1 109.5 mm to (118.1, 127.6)
- moved D3 99.5 mm to (158.8, 128.3)
- moved D4 84.6 mm to (143.5, 128.3)
- moved D1 63.8 mm to (151.1, 128.3)
- moved R4 53.5 mm to (108.0, 127.6)
- moved X1 33.6 mm to (139.1, 87.6)
- moved J5 32.5 mm to (73.7, 125.7)
- moved R3 32.4 mm to (119.4, 106.0), turned to 90 degrees
- moved C2 30.1 mm to (85.1, 125.7)
- moved U16 29.3 mm to (94.6, 127.0)
- moved REF** 10.2 mm to (29.2, 128.3)
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Connections:
- U11 pad 27: /BAUD_B -> Net-(JP1-Pad2)
- U14 pad 21: Net-(U14-Pad21) -> /CLK2
- U14 pad 22: Net-(U14-Pad22) -> /CLK2
- X1 pad 4: (no net) -> GND
- X1 pad 5: (no net) -> Net-(U1-Pad3)
- X1 pad 8: Net-(U1-Pad3) -> +5V
Other:
- board size 172.7 x 116.8 mm -> 172.7 x 106.7 mm

Commit message: update all
Parts:
- removed REF** (x4): MountingHole_2.7mm_Pad, MountingHole:MountingHole_2.7mm_Pad
- removed REF**: lcd, lcd_mount:lcd
- added R8: 4.7k, Resistor_THT:R_Axial_DIN0204_L3.6mm_D1.6mm_P5.08mm_Horizontal, F.Cu at (177.8, 123.2)
- C1: footprint Capacitor_THT:CP_Radial_D5.0mm_P2.50mm -> Capacitor_THT:CP_Radial_Tantal_D5.0mm_P2.50mm
- SW1: footprint Connector_PinHeader_2.54mm:PinHeader_1x02_P2.54mm_Vertical -> Button_Switch_THT:SW_PUSH_6mm
- moved SW1 5.36 mm to (67.0, 123.1), turned to -90 degrees
- moved J5 1.92 mm to (75.5, 126.3)
- moved C1 0.06 mm to (118.2, 127.6)
Connections:
- net Net-(U11-Pad7) renamed /DIEO
- J1 pad 2: Net-(J1-Pad2) -> unconnected-(J1-Pin_2-Pad2)
- J2 pad 4: Net-(J2-Pad4) -> unconnected-(J2-Pin_4-Pad4)
- J3 pad 4: Net-(J3-Pad4) -> unconnected-(J3-Pin_4-Pad4)
- U1 pad 8: Net-(U1-Pad8) -> unconnected-(U1B-~{Q}-Pad8)
- U10 pad 10: Net-(U10-Pad10) -> unconnected-(U10-I1d-Pad10)
- U10 pad 11: Net-(U10-Pad11) -> unconnected-(U10-I0d-Pad11)
- U10 pad 9: Net-(U10-Pad9) -> unconnected-(U10-Zd-Pad9)
- U11 pad 10: Net-(U11-Pad10) -> unconnected-(U11-nW/RDYA-Pad10)
- U11 pad 17: Net-(U11-Pad17) -> unconnected-(U11-nRTSA-Pad17)
- U11 pad 30: Net-(U11-Pad30) -> unconnected-(U11-nW/RDYB-Pad30)
- U14 pad 11: Net-(U14-Pad11) -> unconnected-(U14-IEO-Pad11)
- U14 pad 12: Net-(U14-Pad12) -> /nINT
- U17 pad 6: Net-(U17-Pad6) -> unconnected-(U17A-~{Q}-Pad6)
- U17 pad 9: Net-(U17-Pad9) -> unconnected-(U17B-Q-Pad9)
- U18 pad 12: Net-(U18-Pad12) -> unconnected-(U18B-D-Pad12)
- U18 pad 8: Net-(U18-Pad8) -> unconnected-(U18B-~{Q}-Pad8)
- U18 pad 9: Net-(U18-Pad9) -> unconnected-(U18B-Q-Pad9)
- U2 pad 7: Net-(U2-Pad7) -> unconnected-(U2-O7-Pad7)
- U3 pad 23: Net-(U3-Pad23) -> unconnected-(U3-~{BUSACK}-Pad23)
- U3 pad 28: Net-(U3-Pad28) -> unconnected-(U3-~{RFSH}-Pad28)
- U9 pad 36: /nRD -> /nIORQ
- X1 pad 1: Net-(X1-Pad1) -> unconnected-(X1-EN-Pad1)
Other:
- net class Default removed

Commit message: small tweaks to placement
Parts:
- added C20: 0.1uF, Capacitor_THT:C_Disc_D5.0mm_W2.5mm_P5.00mm, F.Cu at (48.3, 96.5)
- added C21: 0.1uF, Capacitor_THT:C_Disc_D5.0mm_W2.5mm_P5.00mm, F.Cu at (153.7, 81.3)
- added H1: MountingHole, MountingHole:MountingHole_4.3mm_M4, F.Cu at (193.0, 30.5)
- added H2: MountingHole, MountingHole:MountingHole_4.3mm_M4, F.Cu at (30.5, 30.5)
- added H3: MountingHole, MountingHole:MountingHole_4.3mm_M4, F.Cu at (30.5, 127.0)
- added H4: MountingHole, MountingHole:MountingHole_4.3mm_M4, F.Cu at (193.0, 127.0)
- moved C3 56.8 mm to (104.1, 121.9), turned to -90 degrees
- moved J5 31.2 mm to (44.3, 127.0)
- moved C2 5.04 mm to (80.0, 125.7)
- moved R4 3.86 mm to (111.8, 127.0), turned to 90 degrees
- moved SW1 3.59 mm to (70.5, 123.8)
- moved U16 3.17 mm to (91.4, 127.0)
- moved J1 2.69 mm to (194.3, 90.2)
- moved J6 2.29 mm to (30.5, 90.2)
Connections:
- J1 pad 2: unconnected-(J1-Pin_2-Pad2) -> GND
Routing:
- added copper zone on In2.Cu, net +5V
- added copper zone on In1.Cu, net GND

Commit message: demo routing, highlight high current nets
Routing:
- net /A0: track 0.00 -> 97.5 mm, vias 0 -> 1
- net /A6: track 0.00 -> 97.1 mm, vias 0 -> 3
- net /A1: track 0.00 -> 97.0 mm, vias 0 -> 1
- net /A7: track 0.00 -> 96.8 mm, vias 0 -> 3
- net /A3: track 0.00 -> 96.2 mm, vias 0 -> 1
- net /A2: track 0.00 -> 96.1 mm, vias 0 -> 1
- net /A4: track 0.00 -> 95.7 mm, vias 0 -> 1
- net /A5: track 0.00 -> 95.0 mm, vias 0 -> 1
- net /A8: track 0.00 -> 93.3 mm, vias 0 -> 4
- net /A12: track 0.00 -> 67.5 mm, vias 0 -> 1
- net /A9: track 0.00 -> 62.3 mm, vias 0 -> 2
- net /D0: track 0.00 -> 57.9 mm, vias 0 -> 1
- net /D5: track 0.00 -> 57.4 mm, vias 0 -> 2
- net /A13: track 0.00 -> 55.5 mm, vias 0 -> 2
- net /D6: track 0.00 -> 55.0 mm, vias 0 -> 1
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Other:
- rule pad_to_mask_clearance: 0.051 -> 0

Commit message: updating
Parts:
- U1, U12, U13, U15, U17, U18, U6: footprint Package_DIP:DIP-14_W7.62mm_LongPads -> Package_DIP:DIP-14_W7.62mm
- U10, U2, U5, U7: footprint Package_DIP:DIP-16_W7.62mm_LongPads -> Package_DIP:DIP-16_W7.62mm
- U11, U9: footprint Package_DIP:DIP-40_W15.24mm_Socket_LongPads -> Package_DIP:DIP-40_W15.24mm
- U14: footprint Package_DIP:DIP-28_W15.24mm_LongPads -> Package_DIP:DIP-28_W15.24mm
- U3: footprint Package_DIP:DIP-40_W15.24mm_LongPads -> Package_DIP:DIP-40_W15.24mm
- U8: footprint Package_DIP:DIP-32_W15.24mm_LongPads -> Package_DIP:DIP-32_W15.24mm
Routing:
- net /A0: track 97.5 -> 0.00 mm, vias 1 -> 0
- net /A6: track 97.1 -> 0.00 mm, vias 3 -> 0
- net /A1: track 97.0 -> 0.00 mm, vias 1 -> 0
- net /A7: track 96.8 -> 0.00 mm, vias 3 -> 0
- net /A3: track 96.2 -> 0.00 mm, vias 1 -> 0
- net /A2: track 96.1 -> 0.00 mm, vias 1 -> 0
- net /A4: track 95.7 -> 0.00 mm, vias 1 -> 0
- net /A5: track 95.0 -> 0.00 mm, vias 1 -> 0
- net /A8: track 93.3 -> 0.00 mm, vias 4 -> 0
- net /A12: track 67.5 -> 0.00 mm, vias 1 -> 0
- net /A9: track 62.3 -> 0.00 mm, vias 2 -> 0
- net /D5: track 57.4 -> 0.00 mm, vias 2 -> 0
- net /A13: track 55.5 -> 0.00 mm, vias 2 -> 0
- net /D6: track 55.0 -> 0.00 mm, vias 1 -> 0
- net /D4: track 55.0 -> 0.00 mm
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