File: hardware/cpu/cpu.kicad_sch (KiCad schematic)
At the start: 58 parts, among them J1 Conn_02x20_Odd_Even, J2 Conn_01x06, J3 Conn_01x06, J4 Conn_02x05_Odd_Even, J5 Conn_01x02, J6 Conn_02x20_Odd_Even, SW1 SW_Push, U1 74AS74, U10 74LS157, U11 Z80-DART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

Commit message: update all
Parts:
- C1: footprint Capacitor_SMD:C_0805_2012Metric -> Capacitor_THT:CP_Radial_Tantal_D5.0mm_P2.50mm
- R6: footprint Resistor_THT:R_Axial_DIN0918_L18.0mm_D9.0mm_P22.86mm_Horizontal -> Resistor_THT:R_Axial_DIN0204_L3.6mm_D1.6mm_P5.08mm_Horizontal

Commit message: small tweaks to placement
Parts:
- added C20, C21: 0.1uF, Capacitor_THT:C_Disc_D5.0mm_W2.5mm_P5.00mm, symbol Device:C
- added H1, H2, H3, H4: MountingHole, MountingHole:MountingHole_4.3mm_M4, symbol Mechanical:MountingHole
Connections:
- net +5V: now also C20.1, C21.1
- net GND: now also J1.2 (Pin_2), C20.2, C21.2
Other:
- moved on the sheet: C10, C11, C12, C13, C14, C15, C16, C17, C18, C19, C2, C3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

Commit message: updating
Parts:
- removed J6: Conn_02x20_Odd_Even, Connector_PinHeader_2.54mm:PinHeader_2x20_P2.54mm_Vertical, symbol Connector_Generic:Conn_02x20_Odd_Even
- added J6: Conn_02x25_Odd_Even, symbol Connector_Generic:Conn_02x25_Odd_Even
- U1, U12, U13, U15, U17, U18, U6: footprint Package_DIP:DIP-14_W7.62mm_LongPads -> Package_DIP:DIP-14_W7.62mm
- U10, U2, U5, U7: footprint Package_DIP:DIP-16_W7.62mm_LongPads -> Package_DIP:DIP-16_W7.62mm
- U11, U9: footprint Package_DIP:DIP-40_W15.24mm_Socket_LongPads -> Package_DIP:DIP-40_W15.24mm
- U14: footprint Package_DIP:DIP-28_W15.24mm_LongPads -> Package_DIP:DIP-28_W15.24mm
- U3: footprint Package_DIP:DIP-40_W15.24mm_LongPads -> Package_DIP:DIP-40_W15.24mm
- U8: footprint Package_DIP:DIP-32_W15.24mm_LongPads -> Package_DIP:DIP-32_W15.24mm
Connections:
- net +5V: now also J6.43 (Pin_43), J6.44 (Pin_44)
- net A0: now also J6.9 (Pin_9)
- net A1: now also J6.11 (Pin_11)
- net A10: now also J6.29 (Pin_29)
- net A11: now also J6.31 (Pin_31)
- net A12: now also J6.33 (Pin_33)
- net A13: now also J6.35 (Pin_35)
- net A2: now also J6.13 (Pin_13)
- net A3: now also J6.15 (Pin_15)
- net A4: now also J6.17 (Pin_17)
- net A5: now also J6.19 (Pin_19)
- net A6: now also J6.21 (Pin_21)
- net A7: now also J6.23 (Pin_23)
- net A8: now also J6.25 (Pin_25)
- net A9: now also J6.27 (Pin_27)
- net BANK5: now also J6.37 (Pin_37)
- net BANK6: now also J6.39 (Pin_39)
- net CLK: now also J6.40 (Pin_40)
- net D0: now also J6.10 (Pin_10)
- net D1: now also J6.12 (Pin_12)
- net D2: now also J6.14 (Pin_14)
- net D3: now also J6.16 (Pin_16)
- net D4: now also J6.18 (Pin_18)
- net D5: now also J6.20 (Pin_20)
- net D6: now also J6.22 (Pin_22)
- net D7: now also J6.24 (Pin_24)
- net GND: now also J6.1 (Pin_1), J6.2 (Pin_2), J6.3 (Pin_3), J6.4 (Pin_4), J6.47 (Pin_47), J6.48 (Pin_48), J6.49 (Pin_49), J6.5 (Pin_5), J6.50 (Pin_50), J6.6 (Pin_6)
- net nINT: now also J6.38 (Pin_38)
- net nIO14: now also J6.34 (Pin_34)
- net nIO18: now also J6.36 (Pin_36)
- net nIORQ: now also J6.28 (Pin_28)
- net nM1: now also J6.42 (Pin_42)
- net nMREQ: now also J6.26 (Pin_26)
- net nRD: now also J6.30 (Pin_30)
- net nRST: now also J6.41 (Pin_41)
- net nWR: now also J6.32 (Pin_32)
