File: hardware/lcd_adapter/lcd_adapter.sch (KiCad schematic (older format))
At the start: 1 part

Commit message: Schematic partly done
Parts:
- added J?: DB15_Female, symbol Connector:DB15_Female
- added J?: CMOD-A7, symbol Connector_Generic:Conn_02x24_Counter_Clockwise
- added J?: Conn_01x02_Male, symbol Connector:Conn_01x02_Male
- added J?: Conn_02x14_Odd_Even, symbol Connector_Generic:Conn_02x14_Odd_Even
- added JP?: JPR3, symbol Jumper:Jumper_3_Open
- added R? (x14): R_US, symbol Device:R_US
- J?: CatNo (none) -> 798-FH12-33S-0.5SH55; MfgNo (none) -> FH12-33S-0.5SH(55); Supplier (none) -> Mouser
Connections:
- net labels added: +3.3V, GND, LCD_B0, LCD_B1, LCD_B2, LCD_B3, LCD_B4, LCD_B5, LCD_CLK, LCD_DEN, LCD_DISP, LCD_G0, LCD_G1, LCD_G2, LCD_G3, LCD_G4, LCD_G5, LCD_HS, LCD_R0, LCD_R1, LCD_R2, LCD_R3, LCD_R4, LCD_R5, LCD_REV, LCD_VS, VGA_B0, VGA_B1, VGA_B2, VGA_B3, VGA_G0, VGA_G1, VGA_G2, VGA_G3, VGA_HS, VGA_R0, VGA_R1, VGA_R2, VGA_R3, VGA_VS
- wire segments 9 -> 165
- no-connect marks 0 -> 2
Other:
- note added: "A"
- note added: "CMOD S7 LCD/VGA Adapter"
- note added: "Jumper all for VGA"
- note added: "LCD Panel"
- note added: "PMOD GND\n(to improve signal integrity)"
- note added: "TODO:\n* Computer interface\n* Power supplies: 3.3V (regulator)?\n* 12V for backlight (dimmer)?\n"
- note added: "UPCO Graphics Systems"
- note added: "VGA"
- moved on the sheet: J?

Commit message: working on CPU
Parts:
- added J6: Conn_02x17_Odd_Even, Connector_PinHeader_2.54mm:PinHeader_2x17_P2.54mm_Vertical, symbol Connector_Generic:Conn_02x17_Odd_Even
- added U1, U2, U3: SN74LVCC4245A, Package_SO:SO-24_5.3x15mm_P1.27mm, symbol adapter_symbols:SN74LVCC4245A
- J1: renamed from J?; footprint (none) -> Package_DIP:DIP-48_W15.24mm_Socket_LongPads
- J2: renamed from J?; footprint (none) -> Connector_PinHeader_2.54mm:PinHeader_2x01_P2.54mm_Vertical
- J3: renamed from J?; footprint (none) -> Connector_PinHeader_2.54mm:PinHeader_2x14_P2.54mm_Vertical
- J4: renamed from J?; footprint (none) -> Connector_Dsub:DSUB-15-HD_Female_Horizontal_P2.29x1.98mm_EdgePinOffset9.40mm
- J5: renamed from J?; footprint (none) -> lcd_adapter:FH12-33S-0.5
- JP1: renamed from JP?; footprint (none) -> Connector_PinHeader_2.54mm:PinHeader_1x03_P2.54mm_Vertical
- R1, R5, R9: renamed from R?; value R_US -> 4k; footprint (none) -> Resistor_THT:R_Axial_DIN0414_L11.9mm_D4.5mm_P15.24mm_Horizontal
- R10, R2, R6: renamed from R?; value R_US -> 2k; footprint (none) -> Resistor_THT:R_Axial_DIN0414_L11.9mm_D4.5mm_P15.24mm_Horizontal
- R11, R3, R7: renamed from R?; value R_US -> 1k; footprint (none) -> Resistor_THT:R_Axial_DIN0414_L11.9mm_D4.5mm_P15.24mm_Horizontal
- R12, R4, R8: renamed from R?; value R_US -> 510; footprint (none) -> Resistor_THT:R_Axial_DIN0414_L11.9mm_D4.5mm_P15.24mm_Horizontal
- R13, R14: renamed from R?; value R_US -> 100; footprint (none) -> Resistor_THT:R_Axial_DIN0414_L11.9mm_D4.5mm_P15.24mm_Horizontal
Connections:
- net labels added: +5V, A0, A10, A11, A7, A8, A9, D0, D7, DIR, READ, WRITE, ~OE
- wire segments 165 -> 326
Other:
- note added: "CMOD A7 FPGA Module"
- note added: "CPU Interface"
- moved on the sheet: J1, J2, J3, J4, J5, JP1, R1, R10, R11, R12, R13, R14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
