File: hardware/mc6845/memory.sch (KiCad schematic (older format))
At the start: 7 parts, among them U3 74LS157, U4 74LS157, U5 74LS157, U6 74LS157, U8 74LS245, U9 74LS374

Commit message: Add README, work on bitmap mode
Parts:
- removed U?: CY62256-70PC, Package_DIP:DIP-28_W15.24mm, symbol Memory_RAM:CY62256-70PC
- added U?: AS6C4008-55PCN, Package_DIP:DIP-32_W15.24mm, symbol Memory_RAM:AS6C4008-55PCN
- U3, U4, U5, U6: footprint (none) -> Package_DIP:DIP-16_W7.62mm_Socket_LongPads
- U8, U9: footprint (none) -> Package_DIP:DIP-20_W7.62mm_Socket_LongPads
Connections:
- net labels added: A15, MA15, RA15, RA16, RA17, RA18
- wire segments 137 -> 146
Changed lines of the file:
@@
 F 0 "U5" H 5350 3025 50  0000 C CNN
 F 1 "74LS157" H 5450 2925 50  0000 C CNN
-F 2 "" H 5225 2125 50  0001 C CNN
+F 2 "Package_DIP:DIP-16_W7.62mm_Socket_LongPads" H 5225 2125 50  0001 C CNN
 F 3 "http://www.ti.com/lit/gpn/sn74LS157" H 5225 2125 50  0001 C CNN
 	1    5225 2125
@@
 F 0 "U6" H 5325 5650 50  0000 C CNN
 F 1 "74LS157" H 5450 5550 50  0000 C CNN
-F 2 "" H 5225 4750 50  0001 C CNN
+F 2 "Package_DIP:DIP-16_W7.62mm_Socket_LongPads" H 5225 4750 50  0001 C CNN
 F 3 "http://www.ti.com/lit/gpn/sn74LS157" H 5225 4750 50  0001 C CNN
 	1    5225 4750
@@
 F 0 "U3" H 3475 3025 50  0000 C CNN
 F 1 "74LS157" H 3575 2925 50  0000 C CNN
-F 2 "" H 3350 2125 50  0001 C CNN
+F 2 "Package_DIP:DIP-16_W7.62mm_Socket_LongPads" H 3350 2125 50  0001 C CNN
 F 3 "http://www.ti.com/lit/gpn/sn74LS157" H 3350 2125 50  0001 C CNN
 	1    3350 2125
@@
 F 0 "U4" H 3475 5650 50  0000 C CNN
 F 1 "74LS157" H 3575 5550 50  0000 C CNN
-F 2 "" H 3350 4750 50  0001 C CNN
+F 2 "Package_DIP:DIP-16_W7.62mm_Socket_LongPads" H 3350 4750 50  0001 C CNN
 F 3 "http://www.ti.com/lit/gpn/sn74LS157" H 3350 4750 50  0001 C CNN
 	1    3350 4750
@@
 F 0 "U9" H 9525 5325 50  0000 C CNN
 F 1 "74LS374" H 9625 5225 50  0000 C CNN
-F 2 "" H 9400 4550 50  0001 C CNN
+F 2 "Package_DIP:DIP-20_W7.62mm_Socket_LongPads" H 9400 4550 50  0001 C CNN
 F 3 "http://www.ti.com/lit/gpn/sn74LS374" H 9400 4550 50  0001 C CNN
 	1    9400 4550
@@
 Connection ~ 3350 5750
 $Comp
-L power:+5V #PWR?
+L power:+5V #PWR030
 U 1 1 5F3CCAE2
 P 7350 1650
-F 0 "#PWR?" H 7350 1500 50  0001 C CNN
+F 0 "#PWR030" H 7350 1500 50  0001 C CNN
 F 1 "+5V" H 7365 1823 50  0000 C CNN
 F 2 "" H 7350 1650 50  0001 C CNN
@@
 $EndComp
 $Comp
-L power:+5V #PWR?
+L power:+5V #PWR035
 U 1 1 5F3CCB1A
 P 9550 1650
-F 0 "#PWR?" H 9550 1500 50  0001 C CNN
+F 0 "#PWR035" H 9550 1500 50  0001 C CNN
 F 1 "+5V" H 9565 1823 50  0000 C CNN
 F 2 "" H 9550 1650 50  0001 C CNN
@@
 $EndComp
 $Comp
-L power:+5V #PWR?
+L power:+5V #PWR033
 U 1 1 5F3CCB33
 P 9400 3800
-F 0 "#PWR?" H 9400 3650 50  0001 C CNN
+F 0 "#PWR033" H 9400 3650 50  0001 C CNN
 F 1 "+5V" H 9415 3973 50  0000 C CNN
 F 2 "" H 9400 3800 50  0001 C CNN
@@
 $EndComp
 $Comp
-L power:GND #PWR?
+L power:GND #PWR031
 U 1 1 5F3CCBE9
-P 7350 3975
-F 0 "#PWR?" H 7350 3725 50  0001 C CNN
-F 1 "GND" H 7355 3802 50  0000 C CNN
-F 2 "" H 7350 3975 50  0001 C CNN
-F 3 "" H 7350 3975 50  0001 C CNN
-	1    7350 3975
-	1    0    0    -1
-$EndComp
-$Comp
-L power:GND #PWR?
+P 7350 4075
+F 0 "#PWR031" H 7350 3825 50  0001 C CNN
+F 1 "GND" H 7355 3902 50  0000 C CNN
+F 2 "" H 7350 4075 50  0001 C CNN
+F 3 "" H 7350 4075 50  0001 C CNN
+	1    7350 4075
+	1    0    0    -1
+$EndComp
+$Comp
+L power:GND #PWR036
 U 1 1 5F3CCC02
 P 9550 3250
-F 0 "#PWR?" H 9550 3000 50  0001 C CNN
+F 0 "#PWR036" H 9550 3000 50  0001 C CNN
 F 1 "GND" H 9555 3077 50  0000 C CNN
 F 2 "" H 9550 3250 50  0001 C CNN
@@
 $EndComp
 $Comp
-L power:GND #PWR?
+L power:GND #PWR034
 U 1 1 5F3CCC1B
 P 9400 5450
-F 0 "#PWR?" H 9400 5200 50  0001 C CNN
+F 0 "#PWR034" H 9400 5200 50  0001 C CNN
 F 1 "GND" H 9405 5277 50  0000 C CNN
 F 2 "" H 9400 5450 50  0001 C CNN
@@
 MMUX
 Wire Wire Line
-	7350 3975 7350 3550
+	7350 4075 7350 3950
 Wire Wire Line
 	7350 1650 7350 1750
-$Comp
-L Memory_RAM:CY62256-70PC U?
-U 1 1 5F56E878
-P 7350 2650
-F 0 "U?" H 7350 3731 50  0000 C CNN
-F 1 "CY62256-70PC" H 7350 3640 50  0000 C CNN
-F 2 "Package_DIP:DIP-28_W15.24mm" H 7350 2550 50  0001 C CNN
-F 3 "https://ecee.colorado.edu/~mcclurel/Cypress_SRAM_CY62256.pdf" H 7350 2550 50  0001 C CNN
-	1    7350 2650
-	1    0    0    -1
-$EndComp
-Wire Wire Line
-	7850 2850 8125 2850
+Wire Wire Line
+	7950 2850 8125 2850
 Wire Wire Line
 	7850 3050 8125 3050
@@
 F 0 "U8" H 9675 3250 50  0000 C CNN
 F 1 "74LS245" H 9775 3150 50  0000 C CNN
-F 2 "" H 9550 2450 50  0001 C CNN
+F 2 "Package_DIP:DIP-20_W7.62mm_Socket_LongPads" H 9550 2450 50  0001 C CNN
 F 3 "http://www.ti.com/lit/gpn/sn74LS245" H 9550 2450 50  0001 C CNN
 	1    9550 2450
@@
 CCLK
 $Comp
-L power:GND #PWR?
+L power:GND #PWR032
 U 1 1 5F6167B7
 P 8125 2850
-F 0 "#PWR?" H 8125 2600 50  0001 C CNN
-F 1 "GND" H 7975 2800 50  0000 C CNN
+F 0 "#PWR032" H 8125 2600 50  0001 C CNN
+F 1 "GND" H 8125 2925 50  0000 C CNN
 F 2 "" H 8125 2850 50  0001 C CNN
 F 3 "" H 8125 2850 50  0001 C CNN
@@
 	1    0    0    -1
 $EndComp
+$Comp
+L Memory_RAM:AS6C4008-55PCN U?
+U 1 1 5FD424F6
+P 7350 2850
+F 0 "U?" H 7350 4131 50  0000 C CNN
+F 1 "AS6C4008-55PCN" H 7350 4040 50  0000 C CNN
+F 2 "Package_DIP:DIP-32_W15.24mm" H 7350 2950 50  0001 C CNN
+F 3 "https://www.alliancememory.com/wp-content/uploads/pdf/AS6C4008.pdf" H 7350 2950 50  0001 C CNN
+	1    7350 2850
+	1    0    0    -1
+$EndComp
+Wire Wire Line
+	7950 2850 7950 2950
+Wire Wire Line
+	7950 2950 7850 2950
+Wire Wire Line
+	6850 3450 6450 3450
+Wire Wire Line
+	6850 3550 6450 3550
+Wire Wire Line
+	6850 3650 6450 3650
+Wire Wire Line
+	6850 3750 6450 3750
+Text Label 6500 3450 0    50   ~ 0
+RA15
+Text Label 6500 3550 0    50   ~ 0
+RA16
+Text Label 6500 3650 0    50   ~ 0
+RA17
+Text Label 6500 3750 0    50   ~ 0
+RA18
+Wire Wire Line
+	3850 5050 4150 5050
+Wire Wire Line
+	2850 5050 2575 5050
+Wire Wire Line
+	2850 5150 2575 5150
+Text Label 3925 5050 0    50   ~ 0
+RA15
+Text Label 2625 5050 0    50   ~ 0
+MA15
+Text Label 2625 5150 0    50   ~ 0
+A15
 $EndSCHEMATC

Commit message: working on memory
Connections:
- net labels added: A[15..0], MA[15..0], RA[18..16]
- net labels removed: A[13..0], MA[13..0]
Changed lines of the file:
@@
 $EndComp
 Text HLabel 1350 1525 0    50   Input ~ 0
-MA[13..0]
+MA[15..0]
 Text HLabel 1350 1750 0    50   Input ~ 0
-A[13..0]
+A[15..0]
 Wire Wire Line
 	7850 1950 8275 1950
@@
 	1350 1750 1850 1750
 Text Label 1800 1525 2    50   ~ 0
-MA[13..0]
+MA[15..0]
 Text Label 1800 1750 2    50   ~ 0
-A[13..0]
+A[15..0]
 Text HLabel 10800 4050 2    50   Output ~ 0
 LD[7..0]
@@
 U 1 1 5FD424F6
 P 7350 2850
-F 0 "U?" H 7350 4131 50  0000 C CNN
-F 1 "AS6C4008-55PCN" H 7350 4040 50  0000 C CNN
+F 0 "U?" H 7475 4050 50  0000 C CNN
+F 1 "AS6C4008-55PCN" H 7775 3950 50  0000 C CNN
 F 2 "Package_DIP:DIP-32_W15.24mm" H 7350 2950 50  0001 C CNN
 F 3 "https://www.alliancememory.com/wp-content/uploads/pdf/AS6C4008.pdf" H 7350 2950 50  0001 C CNN
@@
 Text Label 2625 5150 0    50   ~ 0
 A15
+Text HLabel 1350 1325 0    50   Input ~ 0
+RA[18..16]
+Wire Bus Line
+	1350 1325 1850 1325
+Text Label 1800 1325 2    50   ~ 0
+RA[18..16]
 $EndSCHEMATC

Commit message: memory
Parts:
- added U?: 74LS157, Package_DIP:DIP-16_W7.62mm_Socket_LongPads, symbol 74xx:74LS157
Connections:
- net labels added: A16, A17, A18, A[18..0], MA16, MA17, MA18, MA[18..0]
- net labels removed: A[15..0], MA[15..0], RA[18..16]
- wire segments 146 -> 162
- no-connect marks 0 -> 1
Other:
- note added: "512K x 8 multiplexed video RAM\n MMUX = H for CPU access, L for CRTC\n nWE, nOE, DIR, nBE for CPU access\n CCLK latches RAM coutput for display"
- note added: "UPCO Graphic Systems"
- note added: "Video RAM"
- moved on the sheet: U3, U4, U5, U6

Commit message: working on 3D
Parts:
- gave numbers to parts that had none: 2
Changed lines of the file:
@@
 $EndComp
 $Comp
-L Memory_RAM:AS6C4008-55PCN U?
+L Memory_RAM:AS6C4008-55PCN U7
 U 1 1 5FD424F6
 P 7350 2850
-F 0 "U?" H 7475 4050 50  0000 C CNN
+F 0 "U7" H 7475 4050 50  0000 C CNN
 F 1 "AS6C4008-55PCN" H 7775 3950 50  0000 C CNN
 F 2 "Package_DIP:DIP-32_W15.24mm" H 7350 2950 50  0001 C CNN
@@
 P 3300 6400
 AR Path="/5FD6FCD7" Ref="U?"  Part="1"
-AR Path="/5F3BFE79/5FD6FCD7" Ref="U?"  Part="1"
-F 0 "U?" H 3425 7300 50  0000 C CNN
+AR Path="/5F3BFE79/5FD6FCD7" Ref="U2"  Part="1"
+F 0 "U2" H 3425 7300 50  0000 C CNN
 F 1 "74LS157" H 3525 7200 50  0000 C CNN
 F 2 "Package_DIP:DIP-16_W7.62mm_Socket_LongPads" H 3300 6400 50  0001 C CNN
@@
 A18
 $Comp
-L power:+5V #PWR?
+L power:+5V #PWR0109
 U 1 1 5FD6FF5D
 P 3300 5500
-F 0 "#PWR?" H 3300 5350 50  0001 C CNN
+F 0 "#PWR0109" H 3300 5350 50  0001 C CNN
 F 1 "+5V" H 3150 5550 50  0000 C CNN
 F 2 "" H 3300 5500 50  0001 C CNN
@@
 $EndComp
 $Comp
-L power:GND #PWR?
+L power:GND #PWR0110
 U 1 1 5FD6FF67
 P 3300 7400
-F 0 "#PWR?" H 3300 7150 50  0001 C CNN
+F 0 "#PWR0110" H 3300 7150 50  0001 C CNN
 F 1 "GND" H 3305 7227 50  0000 C CNN
 F 2 "" H 3300 7400 50  0001 C CNN
@@
 	2600 6700 2800 6700
 $Comp
-L power:GND #PWR?
+L power:GND #PWR0111
 U 1 1 5FDA8AE7
 P 2500 6700
-F 0 "#PWR?" H 2500 6450 50  0001 C CNN
+F 0 "#PWR0111" H 2500 6450 50  0001 C CNN
 F 1 "GND" H 2350 6650 50  0000 C CNN
 F 2 "" H 2500 6700 50  0001 C CNN

Commit message: memory wiring
Parts:
- removed U2: 74LS157, Package_DIP:DIP-16_W7.62mm_Socket_LongPads, symbol 74xx:74LS157
Connections:
- net labels added: A[15..0], MA[15..0], PAGE0, PAGE1, PAGE2, PAGE[0..2]
- net labels removed: A16, A17, A18, A[18..0], MA16, MA17, MA18, MA[18..0], RA16, RA17, RA18
- wire segments 162 -> 146
- no-connect marks 1 -> 0
Changed lines of the file:
@@
 	1    0    0    -1
 $EndComp
-Text HLabel 1350 1525 0    50   Input ~ 0
-MA[18..0]
+Text HLabel 1350 1550 0    50   Input ~ 0
+MA[15..0]
 Text HLabel 1350 1750 0    50   Input ~ 0
-A[18..0]
+A[15..0]
 Wire Wire Line
 	7850 1950 8275 1950
@@
 D[7..0]
 Wire Bus Line
-	1350 1525 1850 1525
+	1350 1550 1850 1550
 Wire Bus Line
 	1350 1750 1850 1750
-Text Label 1800 1525 2    50   ~ 0
-MA[18..0]
+Text Label 1800 1550 2    50   ~ 0
+MA[15..0]
 Text Label 1800 1750 2    50   ~ 0
-A[18..0]
+A[15..0]
 Text HLabel 10800 4050 2    50   Output ~ 0
 LD[7..0]
@@
 Text Label 2525 4700 0    50   ~ 0
 MMUX
-Text HLabel 1350 1975 0    50   Input ~ 0
-MMUX
-Wire Wire Line
-	1350 1975 1850 1975
-Text Label 1500 1975 0    50   ~ 0
+Text HLabel 1350 1950 0    50   Input ~ 0
+MMUX
+Wire Wire Line
+	1350 1950 1850 1950
+Text Label 1500 1950 0    50   ~ 0
 MMUX
 Wire Wire Line
@@
 Text Label 8400 4950 0    50   ~ 0
 CCLK
-Text HLabel 1350 2375 0    50   Input ~ 0
+Text HLabel 1350 2350 0    50   Input ~ 0
 nOE
 Wire Wire Line
-	1350 2375 1850 2375
-Text Label 1500 2375 0    50   ~ 0
+	1350 2350 1850 2350
+Text Label 1500 2350 0    50   ~ 0
 nOE
-Text HLabel 1350 2575 0    50   Input ~ 0
+Text HLabel 1350 2550 0    50   Input ~ 0
 nWE
 Wire Wire Line
-	1350 2575 1850 2575
-Text Label 1500 2575 0    50   ~ 0
+	1350 2550 1850 2550
+Text Label 1500 2550 0    50   ~ 0
 nWE
-Text HLabel 1350 2775 0    50   Input ~ 0
+Text HLabel 1350 2750 0    50   Input ~ 0
 DIR
 Wire Wire Line
-	1350 2775 1850 2775
-Text Label 1500 2775 0    50   ~ 0
+	1350 2750 1850 2750
+Text Label 1500 2750 0    50   ~ 0
 DIR
-Text HLabel 1350 2975 0    50   Input ~ 0
+Text HLabel 1350 2950 0    50   Input ~ 0
 nBE
 Wire Wire Line
-	1350 2975 1850 2975
-Text Label 1500 2975 0    50   ~ 0
+	1350 2950 1850 2950
+Text Label 1500 2950 0    50   ~ 0
 nBE
-Text HLabel 1350 3175 0    50   Input ~ 0
+Text HLabel 1350 3150 0    50   Input ~ 0
 CCLK
 Wire Wire Line
-	1350 3175 1850 3175
-Text Label 1500 3175 0    50   ~ 0
+	1350 3150 1850 3150
+Text Label 1500 3150 0    50   ~ 0
 CCLK
 $Comp
@@
 RA15
 Text Label 6500 3550 0    50   ~ 0
-RA16
+PAGE0
 Text Label 6500 3650 0    50   ~ 0
-RA17
+PAGE1
 Text Label 6500 3750 0    50   ~ 0
-RA18
+PAGE2
 Wire Wire Line
 	3800 4400 4100 4400
@@
 Text Label 2575 4500 0    50   ~ 0
 A15
-$Comp
-L 74xx:74LS157 U?
-U 1 1 5FD6FCD7
-P 3300 6400
-AR Path="/5FD6FCD7" Ref="U?"  Part="1"
-AR Path="/5F3BFE79/5FD6FCD7" Ref="U2"  Part="1"
-F 0 "U2" H 3425 7300 50  0000 C CNN
-F 1 "74LS157" H 3525 7200 50  0000 C CNN
-F 2 "Package_DIP:DIP-16_W7.62mm_Socket_LongPads" H 3300 6400 50  0001 C CNN
-F 3 "http://www.ti.com/lit/gpn/sn74LS157" H 3300 6400 50  0001 C CNN
-	1    3300 6400
-	1    0    0    -1
-$EndComp
-Wire Wire Line
-	3800 5800 4100 5800
-Wire Wire Line
-	3800 6100 4100 6100
-Wire Wire Line
-	3800 6400 4100 6400
-Text Label 3850 5800 0    50   ~ 0
-RA16
-Text Label 3850 6100 0    50   ~ 0
-RA17
-Text Label 3850 6400 0    50   ~ 0
-RA18
-Wire Wire Line
-	2525 5800 2800 5800
-Wire Wire Line
-	2525 5900 2800 5900
-Wire Wire Line
-	2525 6100 2800 6100
-Wire Wire Line
-	2525 6200 2800 6200
-Wire Wire Line
-	2525 6400 2800 6400
-Wire Wire Line
-	2525 6500 2800 6500
-Text Label 2575 5800 0    50   ~ 0
-MA16
-Text Label 2575 5900 0    50   ~ 0
-A16
-Text Label 2575 6100 0    50   ~ 0
-MA17
-Text Label 2575 6200 0    50   ~ 0
-A17
-Text Label 2575 6400 0    50   ~ 0
-MA18
-Text Label 2575 6500 0    50   ~ 0
-A18
-$Comp
-L power:+5V #PWR0109
-U 1 1 5FD6FF5D
-P 3300 5500
-F 0 "#PWR0109" H 3300 5350 50  0001 C CNN
-F 1 "+5V" H 3150 5550 50  0000 C CNN
-F 2 "" H 3300 5500 50  0001 C CNN
-F 3 "" H 3300 5500 50  0001 C CNN
-	1    3300 5500
-	1    0    0    -1
-$EndComp
-$Comp
-L power:GND #PWR0110
-U 1 1 5FD6FF67
-P 3300 7400
-F 0 "#PWR0110" H 3300 7150 50  0001 C CNN
-F 1 "GND" H 3305 7227 50  0000 C CNN
-F 2 "" H 3300 7400 50  0001 C CNN
-F 3 "" H 3300 7400 50  0001 C CNN
-	1    3300 7400
-	1    0    0    -1
-$EndComp
-Wire Wire Line
-	3300 7400 2800 7400
-Wire Wire Line
-	2800 7400 2800 7100
-Connection ~ 3300 7400
-Wire Wire Line
-	2800 7000 2525 7000
-Text Label 2525 7000 0    50   ~ 0
-MMUX
-NoConn ~ 3800 6700
-Wire Wire Line
-	2800 6800 2600 6800
-Wire Wire Line
-	2600 6800 2600 6700
-Wire Wire Line
-	2600 6700 2800 6700
-$Comp
-L power:GND #PWR0111
-U 1 1 5FDA8AE7
-P 2500 6700
-F 0 "#PWR0111" H 2500 6450 50  0001 C CNN
-F 1 "GND" H 2350 6650 50  0000 C CNN
-F 2 "" H 2500 6700 50  0001 C CNN
-F 3 "" H 2500 6700 50  0001 C CNN
-	1    2500 6700
-	1    0    0    -1
-$EndComp
-Wire Wire Line
-	2500 6700 2600 6700
-Connection ~ 2600 6700
 Text Notes 7050 6750 0    100  ~ 0
 UPCO Graphic Systems
@@
 Text Notes 6550 1100 0    75   ~ 0
 512K x 8 multiplexed video RAM\n  MMUX = H for CPU access, L for CRTC\n  nWE, nOE, DIR, nBE for CPU access\n  CCLK latches RAM coutput for display
+Wire Bus Line
+	1850 3350 1350 3350
+Text Label 1450 3350 0    50   ~ 0
+PAGE[0..2]
+Text HLabel 1350 3350 0    50   Input ~ 0
+PAGE[0..2]
 $EndSCHEMATC

Commit message: working
Parts:
- removed U4: 74LS157, Package_DIP:DIP-16_W7.62mm_Socket_LongPads, symbol 74xx:74LS157
- removed U7: AS6C4008-55PCN, Package_DIP:DIP-32_W15.24mm, symbol Memory_RAM:AS6C4008-55PCN
- added U? (x2): 74LS32, symbol 74xx:74LS32
- added U?: 74LS08, symbol 74xx:74LS08
- added U?: 74LS04, symbol 74xx:74LS04
- added U?: AS6C6264, Package_DIP:DIP-28_W15.24mm, symbol video_symbols:AS6C6264
Connections:
- net labels added: A[11..0], MA[11..0], ~OE, ~RD, ~VMEM, ~WE, ~WR
- net labels removed: A12, A13, A14, A15, A[15..0], MA12, MA13, MA14, MA15, MA[15..0], MMUX, PAGE0, PAGE1, PAGE2, PAGE[0..2], RA0, RA1, RA10, RA11, RA12, RA13, RA14, RA15, RA2, RA3, RA4, RA5, RA6, RA7, RA8, RA9, nBE
- wire segments 146 -> 153
Other:
- note added: "4K Video RAM"
- note added: "8K x 8 VIDEO RAM (4K used)"
- note added: "CHARACTER CLOCK"
- note added: "CPU ACCESS BUFFER"
- note added: "CPU ADDRESS"
- note added: "CRTC REFRESH ADDRESS"
- note added: "VIDEO DATA LATCH"
- note added: "~VMEM~ = Video RAM address * ~MREQ"
- note removed: "512K x 8 multiplexed video RAM\n MMUX = H for CPU access, L for CRTC\n nWE, nOE, DIR, nBE for CPU access\n CCLK latches RAM coutput for display"
- note removed: "Video RAM"
- moved on the sheet: U3, U5, U6, U9

Commit message: working on layout
Parts:
- U2, U4, U5: renamed from U?; footprint (none) -> Package_DIP:DIP-14_W7.62mm_Socket_LongPads
- gave numbers to parts that had none: 1
- renumbered U5 to U14, U6 to U15, U3 to U16, U9 to U18, U8 to U19
Changed lines of the file:
@@
 P 4750 1700
 AR Path="/5F3C002B" Ref="U?"  Part="1"
-AR Path="/5F3BFE79/5F3C002B" Ref="U5"  Part="1"
-F 0 "U5" H 4875 2600 50  0000 C CNN
+AR Path="/5F3BFE79/5F3C002B" Ref="U14"  Part="1"
+F 0 "U14" H 4875 2600 50  0000 C CNN
 F 1 "74LS157" H 4975 2500 50  0000 C CNN
 F 2 "Package_DIP:DIP-16_W7.62mm_Socket_LongPads" H 4750 1700 50  0001 C CNN
@@
 P 4750 3850
 AR Path="/5F3C49F8" Ref="U?"  Part="1"
-AR Path="/5F3BFE79/5F3C49F8" Ref="U6"  Part="1"
-F 0 "U6" H 4850 4750 50  0000 C CNN
+AR Path="/5F3BFE79/5F3C49F8" Ref="U15"  Part="1"
+F 0 "U15" H 4850 4750 50  0000 C CNN
 F 1 "74LS157" H 4975 4650 50  0000 C CNN
 F 2 "Package_DIP:DIP-16_W7.62mm_Socket_LongPads" H 4750 3850 50  0001 C CNN
@@
 P 4750 6300
 AR Path="/5F3C5917" Ref="U?"  Part="1"
-AR Path="/5F3BFE79/5F3C5917" Ref="U3"  Part="1"
-F 0 "U3" H 4875 7200 50  0000 C CNN
+AR Path="/5F3BFE79/5F3C5917" Ref="U16"  Part="1"
+F 0 "U16" H 4875 7200 50  0000 C CNN
 F 1 "74LS157" H 4975 7100 50  0000 C CNN
 F 2 "Package_DIP:DIP-16_W7.62mm_Socket_LongPads" H 4750 6300 50  0001 C CNN
@@
 MA11
 $Comp
-L 74xx:74LS374 U9
+L 74xx:74LS374 U18
 U 1 1 5F3C8C42
 P 9400 5050
-F 0 "U9" H 9525 5825 50  0000 C CNN
+F 0 "U18" H 9525 5825 50  0000 C CNN
 F 1 "74LS374" H 9625 5725 50  0000 C CNN
 F 2 "Package_DIP:DIP-20_W7.62mm_Socket_LongPads" H 9400 5050 50  0001 C CNN
@@
 LD7
 $Comp
-L power:GND #PWR0101
+L power:GND #PWR031
 U 1 1 5F43C851
 P 4750 7300
-F 0 "#PWR0101" H 4750 7050 50  0001 C CNN
+F 0 "#PWR031" H 4750 7050 50  0001 C CNN
 F 1 "GND" H 4900 7325 50  0000 C CNN
 F 2 "" H 4750 7300 50  0001 C CNN
@@
 $EndComp
 $Comp
-L power:+5V #PWR0102
+L power:+5V #PWR030
 U 1 1 5F441583
 P 4750 5400
-F 0 "#PWR0102" H 4750 5250 50  0001 C CNN
+F 0 "#PWR030" H 4750 5250 50  0001 C CNN
 F 1 "+5V" H 4765 5573 50  0000 C CNN
 F 2 "" H 4750 5400 50  0001 C CNN
@@
 $EndComp
 $Comp
-L power:+5V #PWR0103
+L power:+5V #PWR026
 U 1 1 5F441609
 P 4750 800
-F 0 "#PWR0103" H 4750 650 50  0001 C CNN
+F 0 "#PWR026" H 4750 650 50  0001 C CNN
 F 1 "+5V" H 4765 973 50  0000 C CNN
 F 2 "" H 4750 800 50  0001 C CNN
@@
 $EndComp
 $Comp
-L power:+5V #PWR0105
+L power:+5V #PWR028
 U 1 1 5F4416F3
 P 4750 2950
-F 0 "#PWR0105" H 4750 2800 50  0001 C CNN
+F 0 "#PWR028" H 4750 2800 50  0001 C CNN
 F 1 "+5V" H 4575 3000 50  0000 C CNN
 F 2 "" H 4750 2950 50  0001 C CNN
@@
 $EndComp
 $Comp
-L power:GND #PWR0106
+L power:GND #PWR027
 U 1 1 5F44174C
 P 4750 2700
-F 0 "#PWR0106" H 4750 2450 50  0001 C CNN
+F 0 "#PWR027" H 4750 2450 50  0001 C CNN
 F 1 "GND" H 4875 2725 50  0000 C CNN
 F 2 "" H 4750 2700 50  0001 C CNN
@@
 Connection ~ 4750 7300
 $Comp
-L power:GND #PWR0108
+L power:GND #PWR029
 U 1 1 5F44B7BF
 P 4750 4850
-F 0 "#PWR0108" H 4750 4600 50  0001 C CNN
+F 0 "#PWR029" H 4750 4600 50  0001 C CNN
 F 1 "GND" H 4755 4677 50  0000 C CNN
 F 2 "" H 4750 4850 50  0001 C CNN
@@
 Connection ~ 4750 4850
 $Comp
-L power:+5V #PWR030
+L power:+5V #PWR033
 U 1 1 5F3CCAE2
 P 7200 1650
-F 0 "#PWR030" H 7200 1500 50  0001 C CNN
+F 0 "#PWR033" H 7200 1500 50  0001 C CNN
 F 1 "+5V" H 7215 1823 50  0000 C CNN
 F 2 "" H 7200 1650 50  0001 C CNN
@@
 $EndComp
 $Comp
-L power:+5V #PWR035
+L power:+5V #PWR038
 U 1 1 5F3CCB1A
 P 9550 1650
-F 0 "#PWR035" H 9550 1500 50  0001 C CNN
+F 0 "#PWR038" H 9550 1500 50  0001 C CNN
 F 1 "+5V" H 9565 1823 50  0000 C CNN
 F 2 "" H 9550 1650 50  0001 C CNN
@@
 $EndComp
 $Comp
-L power:+5V #PWR033
+L power:+5V #PWR036
 U 1 1 5F3CCB33
 P 9400 4300
-F 0 "#PWR033" H 9400 4150 50  0001 C CNN
+F 0 "#PWR036" H 9400 4150 50  0001 C CNN
 F 1 "+5V" H 9415 4473 50  0000 C CNN
 F 2 "" H 9400 4300 50  0001 C CNN
@@
 $EndComp
 $Comp
-L power:GND #PWR031
+L power:GND #PWR034
 U 1 1 5F3CCBE9
 P 7200 3675
-F 0 "#PWR031" H 7200 3425 50  0001 C CNN
+F 0 "#PWR034" H 7200 3425 50  0001 C CNN
 F 1 "GND" H 7205 3502 50  0000 C CNN
 F 2 "" H 7200 3675 50  0001 C CNN
@@
 $EndComp
 $Comp
-L power:GND #PWR036
+L power:GND #PWR039
 U 1 1 5F3CCC02
 P 9550 3250
-F 0 "#PWR036" H 9550 3000 50  0001 C CNN
+F 0 "#PWR039" H 9550 3000 50  0001 C CNN
 F 1 "GND" H 9555 3077 50  0000 C CNN
 F 2 "" H 9550 3250 50  0001 C CNN
@@
 $EndComp
 $Comp
-L power:GND #PWR034
+L power:GND #PWR037
 U 1 1 5F3CCC1B
 P 9400 5950
-F 0 "#PWR034" H 9400 5700 50  0001 C CNN
+F 0 "#PWR037" H 9400 5700 50  0001 C CNN
 F 1 "GND" H 9405 5777 50  0000 C CNN
 F 2 "" H 9400 5950 50  0001 C CNN
@@
 DIR
 $Comp
-L 74xx:74LS245 U8
+L 74xx:74LS245 U19
 U 1 1 5F3C8B19
 P 9550 2450
-F 0 "U8" H 9675 3250 50  0000 C CNN
+F 0 "U19" H 9675 3250 50  0000 C CNN
 F 1 "74LS245" H 9775 3150 50  0000 C CNN
 F 2 "Package_DIP:DIP-20_W7.62mm_Socket_LongPads" H 9550 2450 50  0001 C CNN
@@
 	1150 4000 1650 4000
 $Comp
-L power:GND #PWR032
+L power:GND #PWR035
 U 1 1 5F6167B7
 P 7975 2850
-F 0 "#PWR032" H 7975 2600 50  0001 C CNN
+F 0 "#PWR035" H 7975 2600 50  0001 C CNN
 F 1 "GND" H 7975 2925 50  0000 C CNN
 F 2 "" H 7975 2850 50  0001 C CNN
@@
 4K Video RAM
 $Comp
-L 74xx:74LS32 U?
-U 1 1 613916CD
+L 74xx:74LS32 U2
+U 3 1 613916CD
 P 1850 5850
-F 0 "U?" H 1600 6100 50  0000 C CNN
+F 0 "U2" H 1600 6100 50  0000 C CNN
 F 1 "74LS32" H 1950 6100 50  0000 C CNN
-F 2 "" H 1850 5850 50  0001 C CNN
+F 2 "Package_DIP:DIP-14_W7.62mm_Socket_LongPads" H 1850 5850 50  0001 C CNN
 F 3 "http://www.ti.com/lit/gpn/sn74LS32" H 1850 5850 50  0001 C CNN
-	1    1850 5850
-	1    0    0    -1
-$EndComp
-$Comp
-L 74xx:74LS32 U?
-U 1 1 6139288E
+	3    1850 5850
+	1    0    0    -1
+$EndComp
+$Comp
+L 74xx:74LS32 U2
+U 2 1 6139288E
 P 1850 6450
-F 0 "U?" H 1600 6700 50  0000 C CNN
+F 0 "U2" H 1600 6700 50  0000 C CNN
 F 1 "74LS32" H 1950 6700 50  0000 C CNN
-F 2 "" H 1850 6450 50  0001 C CNN
+F 2 "Package_DIP:DIP-14_W7.62mm_Socket_LongPads" H 1850 6450 50  0001 C CNN
 F 3 "http://www.ti.com/lit/gpn/sn74LS32" H 1850 6450 50  0001 C CNN
-	1    1850 6450
-	1    0    0    -1
-$EndComp
-$Comp
-L 74xx:74LS08 U?
-U 1 1 613970B8
+	2    1850 6450
+	1    0    0    -1
+$EndComp
+$Comp
+L 74xx:74LS08 U5
+U 4 1 613970B8
 P 2700 6900
-F 0 "U?" H 2550 7150 50  0000 C CNN
+F 0 "U5" H 2550 7150 50  0000 C CNN
 F 1 "74LS08" H 2900 7150 50  0000 C CNN
-F 2 "" H 2700 6900 50  0001 C CNN
+F 2 "Package_DIP:DIP-14_W7.62mm_Socket_LongPads" H 2700 6900 50  0001 C CNN
 F 3 "http://www.ti.com/lit/gpn/sn74LS08" H 2700 6900 50  0001 C CNN
-	1    2700 6900
-	1    0    0    -1
-$EndComp
-$Comp
-L 74xx:74LS04 U?
-U 1 1 6139B2A8
+	4    2700 6900
+	1    0    0    -1
+$EndComp
+$Comp
+L 74xx:74LS04 U4
+U 3 1 6139B2A8
 P 1850 7000
-F 0 "U?" H 1850 7317 50  0000 C CNN
+F 0 "U4" H 1850 7317 50  0000 C CNN
 F 1 "74LS04" H 1850 7226 50  0000 C CNN
-F 2 "" H 1850 7000 50  0001 C CNN
+F 2 "Package_DIP:DIP-14_W7.62mm_Socket_LongPads" H 1850 7000 50  0001 C CNN
 F 3 "http://www.ti.com/lit/gpn/sn74LS04" H 1850 7000 50  0001 C CNN
-	1    1850 7000
+	3    1850 7000
 	1    0    0    -1
 $EndComp
@@
 	5250 6600 6100 6600
 $Comp
-L video_symbols:AS6C6264 U?
+L video_symbols:AS6C6264 U17
 U 1 1 6154F446
 P 7200 2650
-F 0 "U?" H 7350 3650 50  0000 C CNN
+F 0 "U17" H 7350 3650 50  0000 C CNN
 F 1 "AS6C6264" H 7500 3550 50  0000 C CNN
 F 2 "Package_DIP:DIP-28_W15.24mm" H 7200 2550 50  0001 C CNN
@@
 	6700 3250 6700 3350
 $Comp
-L power:+5V #PWR?
+L power:+5V #PWR032
 U 1 1 6156DBF2
 P 6550 3350
-F 0 "#PWR?" H 6550 3200 50  0001 C CNN
+F 0 "#PWR032" H 6550 3200 50  0001 C CNN
 F 1 "+5V" H 6565 3523 50  0000 C CNN
 F 2 "" H 6550 3350 50  0001 C CNN
