File: hardware/mc6845/mc6845.kicad_pcb (KiCad board)
At the start: 2 copper layers, 101.6 x 101.6 mm, 19 parts, among them J1 Conn_02x20_Odd_Even, U1 MC6845, U10 AT28C16, U11 74LS32, U12 74LS163, U13 74LS04, U14 74LS08, U15 74LS74, U16 74LS174, U17 74LS165, U2 74LS157, U3 74LS157, U4 74LS157, U5 74LS157, U6 74LS157, U7 AS6C4008-55PCN, U8 74LS245, U9 74LS374, X1 25.175MHz

Commit message: working on layout
Parts:
- removed U10: AT28C16, Package_DIP:DIP-24_W15.24mm_LongPads
- removed U11: 74LS32, Package_DIP:DIP-14_W7.62mm_Socket_LongPads
- removed the U15 at (137.2, 120.0)
- removed the U3 at (95.9, 74.3)
- removed the U4 at (95.9, 87.6)
- removed the U7 at (119.4, 53.3)
- added C1: 0.1uF, Capacitor_THT:C_Disc_D3.0mm_W1.6mm_P2.50mm, F.Cu at (161.6, 102.1)
- added C10: 0.1uF, Capacitor_THT:C_Disc_D3.0mm_W1.6mm_P2.50mm, F.Cu at (166.5, 95.0)
- added C11: 0.1uF, Capacitor_THT:C_Disc_D3.0mm_W1.6mm_P2.50mm, F.Cu at (172.1, 95.0)
- added C12: 0.1uF, Capacitor_THT:C_Disc_D3.0mm_W1.6mm_P2.50mm, F.Cu at (161.1, 72.2)
- added C13: 0.1uF, Capacitor_THT:C_Disc_D3.0mm_W1.6mm_P2.50mm, F.Cu at (161.1, 75.3)
- added C14: 0.1uF, Capacitor_THT:C_Disc_D3.0mm_W1.6mm_P2.50mm, F.Cu at (166.7, 72.2)
- added C15: 0.1uF, Capacitor_THT:C_Disc_D3.0mm_W1.6mm_P2.50mm, F.Cu at (161.1, 78.5)
- added C16: 0.1uF, Capacitor_THT:C_Disc_D3.0mm_W1.6mm_P2.50mm, F.Cu at (166.7, 75.3)
- added C17: 0.1uF, Capacitor_THT:C_Disc_D3.0mm_W1.6mm_P2.50mm, F.Cu at (172.4, 72.2)
- added C2: 0.1uF, Capacitor_THT:C_Disc_D3.0mm_W1.6mm_P2.50mm, F.Cu at (167.3, 104.0)
- added C3: 0.1uF, Capacitor_THT:C_Disc_D3.0mm_W1.6mm_P2.50mm, F.Cu at (160.8, 91.9)
- added C4: 0.1uF, Capacitor_THT:C_Disc_D3.0mm_W1.6mm_P2.50mm, F.Cu at (172.9, 102.4)
- added C5: 10uF, Capacitor_THT:CP_Radial_Tantal_D5.5mm_P5.00mm, F.Cu at (59.7, 115.6)
- added C6: 0.1uF, Capacitor_THT:C_Disc_D3.0mm_W1.6mm_P2.50mm, F.Cu at (160.8, 95.0)
- added C7: 0.1uF, Capacitor_THT:C_Disc_D3.0mm_W1.6mm_P2.50mm, F.Cu at (166.5, 91.9)
- added C8: 0.1uF, Capacitor_THT:C_Disc_D3.0mm_W1.6mm_P2.50mm, F.Cu at (172.1, 91.9)
- added C9: 0.1uF, Capacitor_THT:C_Disc_D3.0mm_W1.6mm_P2.50mm, F.Cu at (177.8, 91.9)
- added H1: MountingHole_Pad, MountingHole:MountingHole_2.7mm_M2.5_DIN965_Pad, F.Cu at (57.8, 50.2)
- added H2: MountingHole_Pad, MountingHole:MountingHole_2.7mm_M2.5_DIN965_Pad, F.Cu at (57.8, 144.1)
- added H3: MountingHole_Pad, MountingHole:MountingHole_2.7mm_M2.5_DIN965_Pad, F.Cu at (151.8, 144.1)
- added H4: MountingHole_Pad, MountingHole:MountingHole_2.7mm_M2.5_DIN965_Pad, F.Cu at (151.8, 50.2)
- added J2: DB15_Female_HighDensity, Connector_Dsub:DSUB-15-HD_Female_Horizontal_P2.29x2.54mm_EdgePinOffset9.40mm, F.Cu at (140.3, 127.0)
- added J3: Conn_01x02, Connector_Molex:Molex_Mini-Fit_Jr_5566-02A_2x01_P4.20mm_Vertical, F.Cu at (61.0, 124.5)
- added U16: 74LS157, Package_DIP:DIP-16_W7.62mm_Socket_LongPads, F.Cu at (94.0, 100.3)
- added U17: AS6C6264, Package_DIP:DIP-28_W15.24mm, F.Cu at (123.2, 88.9)
- added U19: 74LS245, Package_DIP:DIP-20_W7.62mm_Socket_LongPads, F.Cu at (109.2, 55.9)
- added U6: 74LS74, Package_DIP:DIP-14_W7.62mm_Socket_LongPads, F.Cu at (144.8, 101.6)
- J1: footprint Connector_PinHeader_2.54mm:PinHeader_2x20_P2.54mm_Vertical -> Connector_PinSocket_2.54mm:PinSocket_2x20_P2.54mm_Vertical
- U14: value 74LS08 -> 74LS157; footprint Package_DIP:DIP-14_W7.62mm_Socket_LongPads -> Package_DIP:DIP-16_W7.62mm_Socket_LongPads
- U2: value 74LS157 -> 74LS32; footprint Package_DIP:DIP-16_W7.62mm_Socket_LongPads -> Package_DIP:DIP-14_W7.62mm_Socket_LongPads
- U5: value 74LS157 -> 74LS08; footprint Package_DIP:DIP-16_W7.62mm_Socket_LongPads -> Package_DIP:DIP-14_W7.62mm_Socket_LongPads
- U8: value 74LS245 -> 28C64A-15; footprint Package_DIP:DIP-20_W7.62mm_Socket_LongPads -> Package_DIP:DIP-28_W15.24mm
- U9: renamed from U17; value 74LS165 -> 74ALS165
- X1: value 25.175MHz -> MXO45HS-3C-25M1750
- moved U8 90.4 mm to (123.2, 50.8), turned to 0 degrees
- moved U14 79.6 mm to (94.0, 50.8)
- moved X1 77.0 mm to (71.1, 109.2)
- moved U2 49.2 mm to (144.8, 55.9), turned to 0 degrees
- moved U7 46.4 mm to (86.4, 125.7)
- moved U15 38.1 mm to (94.0, 76.2), turned to 0 degrees
- moved U5 35.2 mm to (118.1, 128.3), turned to 0 degrees
- moved U18 15.4 mm to (109.2, 87.6)
- moved U4 14.0 mm to (102.9, 128.3)
- moved U9 5.43 mm to (152.4, 94.6), turned to 180 degrees
- moved U3 2.84 mm to (71.1, 125.7)
- moved J1 2.01 mm to (62.2, 55.9)
- moved U1 1.42 mm to (71.1, 53.3)
- renumbered U6 to U15, U9 to U18, U12 to U3, U13 to U4, U16 to U7
Connections:
- net /~DS0 renamed /~CRTC
- net /~DS3 renamed Net-(J1-Pad35)
- J1 pad 1: Net-(J1-Pad1) -> GND
- J1 pad 19: Net-(J1-Pad19) -> GND
- J1 pad 2: Net-(J1-Pad2) -> GND
- J1 pad 20: Net-(J1-Pad20) -> GND
- J1 pad 31: /~DS1 -> /~VMEM
- J1 pad 33: /~DS2 -> /~RST
- J1 pad 37: /~RST -> Net-(J1-Pad37)
- J1 pad 39: Net-(J1-Pad39) -> GND
- J1 pad 40: Net-(J1-Pad40) -> GND
- U14 pad 1: Net-(U11-Pad3) -> /~VMEM
- U14 pad 10: /VS -> /MA2
- U14 pad 11: (no net) -> /A2
- U14 pad 12: (no net) -> Net-(U14-Pad12)
- U14 pad 13: (no net) -> /MA3
- U14 pad 14: +5V -> /A3
- U14 pad 2: Net-(U14-Pad2) -> /A0
- U14 pad 3: Net-(U14-Pad3) -> /MA0
- U14 pad 4: /HS -> Net-(U14-Pad4)
- U14 pad 5: /HS -> /A1
- U14 pad 6: /HSYNC -> /MA1
- U14 pad 7: GND -> Net-(U14-Pad7)
- U14 pad 8: /VSYNC -> GND
- U14 pad 9: /VS -> Net-(U14-Pad9)
- U15 pad 1: /MEMCPU -> /~VMEM
- U15 pad 10: /A6 -> /MA6
- U15 pad 11: /MA6 -> /A6
- U15 pad 12: /memory/RA7 -> Net-(U15-Pad12)
- U15 pad 13: /A7 -> /MA7
- U15 pad 14: /MA7 -> /A7
- U15 pad 2: /MA4 -> /A4
- U15 pad 3: /A4 -> /MA4
- U15 pad 4: /memory/RA4 -> Net-(U15-Pad4)
- U15 pad 5: /MA5 -> /A5
- U15 pad 6: /A5 -> /MA5
- U15 pad 7: /memory/RA5 -> Net-(U15-Pad7)
- U15 pad 9: /memory/RA6 -> Net-(U15-Pad9)
- U18 pad 13: Net-(U7-Pad18) -> Net-(U17-Pad16)
- U18 pad 14: Net-(U7-Pad19) -> Net-(U17-Pad17)
- U18 pad 17: Net-(U7-Pad20) -> Net-(U17-Pad18)
- U18 pad 18: Net-(U7-Pad21) -> Net-(U17-Pad19)
- U18 pad 19: /memory/LD7 -> /LD7
- U18 pad 3: Net-(U7-Pad13) (its old number) -> Net-(U17-Pad11)
- U18 pad 4: Net-(U7-Pad14) (its old number) -> Net-(U17-Pad12)
- U18 pad 7: Net-(U7-Pad15) (its old number) -> Net-(U17-Pad13)
- U18 pad 8: Net-(U7-Pad17) -> Net-(U17-Pad15)
- U2 pad 1: /MEMCPU -> Net-(U2-Pad1)
- U2 pad 10: /memory/A18 -> /~WR
- U2 pad 11: /memory/MA18 -> (no net)
- U2 pad 12: Net-(U2-Pad12) -> (no net)
- U2 pad 13: GND -> (no net)
- U2 pad 14: GND -> +5V
- U2 pad 2: /memory/MA16 -> Net-(U2-Pad2)
- U2 pad 3: /memory/A16 -> Net-(U2-Pad3)
- U2 pad 4: /memory/RA16 -> /~VMEM
- U2 pad 5: /memory/MA17 -> /~RD
- U2 pad 6: /memory/A17 -> /memory/DIR
- U2 pad 7: /memory/RA17 -> GND
- U2 pad 8: GND -> /memory/~WE
- U2 pad 9: /memory/RA18 -> /~VMEM
- U4 pad 14: (no net) -> +5V
- U4 pad 5: (no net) -> /~VMEM
- U4 pad 6: (no net) -> Net-(U4-Pad6)
- U4 pad 7: (no net) -> GND
- U5 pad 1: /MEMCPU -> Net-(U2-Pad3)
- U5 pad 10: /A2 -> /VS
- U5 pad 11: /MA2 -> /memory/~OE
- U5 pad 12: /memory/RA3 -> /memory/DIR
- U5 pad 13: /A3 -> Net-(U4-Pad6)
- U5 pad 14: /MA3 -> +5V
- U5 pad 2: /MA0 -> Net-(U5-Pad2)
- U5 pad 3: /A0 -> Net-(U5-Pad3)
- U5 pad 4: /memory/RA0 -> /HS
- U5 pad 5: /MA1 -> /HS
- U5 pad 6: /A1 -> /HSYNC
- U5 pad 7: /memory/RA1 -> GND
- U5 pad 8: GND -> /VSYNC
- U5 pad 9: /memory/RA2 -> /VS
- U7 pad 10: Net-(U14-Pad2) -> Net-(U5-Pad2)
- U7 pad 5: Net-(U11-Pad2) -> Net-(U2-Pad2)
- U8 pad 1: /DIR -> (no net)
- U8 pad 10: GND -> /LD0
- U8 pad 11: /D7 -> Net-(U8-Pad11)
- U8 pad 12: /D6 -> Net-(U8-Pad12)
- U8 pad 13: /D5 -> Net-(U8-Pad13)
- U8 pad 14: /D4 -> Net-(U8-Pad14)
- U8 pad 15: /D3 -> Net-(U8-Pad15)
- U8 pad 16: /D2 -> Net-(U8-Pad16)
- U8 pad 17: /D1 -> Net-(U8-Pad17)
- U8 pad 18: /D0 -> Net-(U8-Pad18)
- U8 pad 19: /~MEM_RD -> Net-(U8-Pad19)
- U8 pad 2: Net-(U7-Pad13) (its old number) -> GND
- U8 pad 20: +5V -> GND
- U8 pad 3: Net-(U7-Pad14) (its old number) -> /LD7
- U8 pad 4: Net-(U7-Pad15) (its old number) -> /LD6
- U8 pad 5: Net-(U7-Pad17) -> /LD5
- U8 pad 6: Net-(U7-Pad18) -> /LD4
- U8 pad 7: Net-(U7-Pad19) -> /LD3
- U8 pad 8: Net-(U7-Pad20) -> /LD2
- U8 pad 9: Net-(U7-Pad21) -> /LD1
- U9 pad 11: Net-(U10-Pad9) -> Net-(U8-Pad11)
- U9 pad 12: Net-(U10-Pad10) -> Net-(U8-Pad12)
- U9 pad 13: Net-(U10-Pad11) -> Net-(U8-Pad13)
- U9 pad 14: Net-(U10-Pad13) -> Net-(U8-Pad15)
- U9 pad 16: Net-(U17-Pad16) -> +5V
- U9 pad 3: Net-(U10-Pad14) -> Net-(U8-Pad16)
- U9 pad 4: Net-(U10-Pad15) -> Net-(U8-Pad17)
- U9 pad 5: Net-(U10-Pad16) -> Net-(U8-Pad18)
- U9 pad 6: Net-(U10-Pad17) -> Net-(U8-Pad19)
- U9 pad 9: Net-(U11-Pad1) -> Net-(U2-Pad1)
Other:
- board size 101.6 x 101.6 mm -> 100 x 100 mm

Commit message: started routing
Parts:
- U14, U15, U16, U3, U7, U9: footprint Package_DIP:DIP-16_W7.62mm_Socket_LongPads -> Package_DIP:DIP-16_W7.62mm_Socket
- U18, U19: footprint Package_DIP:DIP-20_W7.62mm_Socket_LongPads -> Package_DIP:DIP-20_W7.62mm_Socket
- U2, U4, U5, U6: footprint Package_DIP:DIP-14_W7.62mm_Socket_LongPads -> Package_DIP:DIP-14_W7.62mm_Socket
- X1: footprint Package_DIP:DIP-8_W7.62mm_LongPads -> Package_DIP:DIP-8_W7.62mm_Socket
- moved C11 97.2 mm to (78.7, 121.9), turned to 180 degrees
- moved C1 90.5 mm to (71.2, 104.1)
- moved C12 89.5 mm to (77.5, 104.1)
- moved C8 83.8 mm to (93.9, 121.9), turned to 180 degrees
- moved C17 73.3 mm to (99.1, 72.4), turned to 180 degrees
- moved C14 64.9 mm to (105.5, 50.8)
- moved C10 63.3 mm to (110.5, 124.5), turned to 180 degrees
- moved C16 57.9 mm to (114.3, 50.8), turned to 180 degrees
- moved C7 51.8 mm to (129.6, 128.3)
- moved C9 50.9 mm to (146.0, 52.1), turned to 180 degrees
- moved C13 32.7 mm to (141.0, 49.5)
- moved C15 25.2 mm to (144.8, 97.8)
- moved C6 23.6 mm to (138.4, 87.6), turned to 180 degrees
- moved C3 10.3 mm to (152.4, 97.8), turned to 180 degrees
- moved J1 2.84 mm to (61.0, 58.4)
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Connections:
- U1 pad 20: Net-(U1-Pad20) -> +5V
Routing:
- net /A0: track 0.00 -> 73.8 mm, vias 0 -> 1
- net /D3: track 0.00 -> 62.3 mm, vias 0 -> 2
- net /A3: track 0.00 -> 52.6 mm, vias 0 -> 1
- net /A2: track 0.00 -> 44.2 mm
- net /A1: track 0.00 -> 36.6 mm
- net /D0: track 0.00 -> 32.4 mm, vias 0 -> 1
- net /D1: track 0.00 -> 32.1 mm, vias 0 -> 1
- net /D2: track 0.00 -> 31.1 mm, vias 0 -> 1
Other:
- net class Default: clearance 0.2 -> 0.127; trace_width 0.25 -> 0.127; via_dia 0.8 -> 0.6096; via_drill 0.4 -> 0.3048
- rule trace_clearance: 0.2 -> 0.127
- rule trace_min: 0.2 -> 0.127
- rule via_min_drill: 0.3 -> 0.3048
- rule via_min_size: 0.4 -> 0.6096

Commit message: RC2014 ideas
Parts:
- added ?: , Pin_Headers:Pin_Header_Straight_1x40, F.Cu at (176.7, 143.0)
- added ?: , Pin_Headers:Pin_Header_Straight_1x10, F.Cu at (217.4, 140.5)
- added ?: , Pin_Headers:Pin_Header_Straight_1x40, F.Cu at (177.7, 67.1)
- added ?: , Pin_Headers:Pin_Header_Straight_1x10, F.Cu at (218.3, 64.6)
- added REF**: DIP-14_W7.62mm_Socket, Package_DIP:DIP-14_W7.62mm_Socket, F.Cu at (256.5, 59.4)
- added REF**: DIP-16_W7.62mm_Socket, Package_DIP:DIP-16_W7.62mm_Socket, F.Cu at (233.4, 59.1)
- added REF**: DIP-16_W7.62mm_Socket, Package_DIP:DIP-16_W7.62mm_Socket, F.Cu at (206.4, 105.7)
- added REF**: DIP-14_W7.62mm_Socket, Package_DIP:DIP-14_W7.62mm_Socket, F.Cu at (270.5, 118.7)
- added REF**: PinSocket_2x12_P2.54mm_Vertical, Connector_PinSocket_2.54mm:PinSocket_2x12_P2.54mm_Vertical, F.Cu at (239.7, 21.3)
- added REF**: PinSocket_2x12_P2.54mm_Vertical, Connector_PinSocket_2.54mm:PinSocket_2x12_P2.54mm_Vertical, F.Cu at (239.1, 97.2)
- moved U4 179.5 mm to (256.5, 35.6), turned to 90 degrees
- moved U3 162.3 mm to (195.6, 21.6)
- moved U5 160.7 mm to (256.5, 46.7), turned to 90 degrees
- moved U7 159.9 mm to (207.6, 21.6)
- moved U1 156.0 mm to (227.0, 44.1), turned to 270 degrees
- moved U8 144.0 mm to (238.4, 137.2), turned to 90 degrees
- moved C4 140.7 mm to (33.2, 85.3)
- moved C2 135.9 mm to (33.3, 81.0)
- moved X1 135.9 mm to (182.6, 31.4)
- moved J2 132.6 mm to (264.2, 79.7)
- moved U18 128.7 mm to (234.3, 117.8), turned to 90 degrees
- moved U19 114.9 mm to (206.1, 117.8), turned to 90 degrees
- moved U14 108.6 mm to (182.6, 113.7), turned to 90 degrees
- moved U6 107.8 mm to (219.7, 24.1)
- moved U9 100.2 mm to (233.4, 35.6), turned to 90 degrees
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Routing:
- net /A0: track 73.8 -> 0.00 mm, vias 1 -> 0
- net /D3: track 62.3 -> 0.00 mm, vias 2 -> 0
- net /A3: track 52.6 -> 0.00 mm, vias 1 -> 0
- net /A2: track 44.2 -> 0.00 mm
- net /A1: track 36.6 -> 0.00 mm
- net /D0: track 32.4 -> 0.00 mm, vias 1 -> 0
- net /D1: track 32.1 -> 0.00 mm, vias 1 -> 0
- net /D2: track 31.1 -> 0.00 mm, vias 1 -> 0
Other:
- board size 100 x 100 mm -> 220 x 128 mm
- net class Default: clearance 0.127 -> 0.1524; trace_width 0.127 -> 0.1778
- rule trace_clearance: 0.127 -> 0.1524
- rule trace_min: 0.127 -> 0.1778
