File: hardware/keyboard/minimal-60-v3/minimal-60-v3.sch (KiCad schematic (older format))
At the start: 137 parts, among them J1 Conn_02x03_Odd_Even, J2 Conn_01x06, K0 KEYSW, K1 KEYSW, K10 KEYSW, K11 KEYSW, K12 KEYSW, K13 KEYSW, K14 KEYSW, K15 KEYSW, K16 KEYSW, K17 KEYSW, K18 KEYSW, K19 KEYSW, K2 KEYSW, K20 KEYSW, K21 KEYSW, K22 KEYSW, K23 KEYSW, K24 KEYSW, K25 KEYSW, K26 KEYSW, K27 KEYSW, K28 KEYSW, K29 KEYSW, K3 KEYSW, K30 KEYSW, K31 KEYSW, K32 KEYSW, K33 KEYSW, K34 KEYSW, K35 KEYSW, K36 KEYSW, K37 KEYSW, K38 KEYSW, K39 KEYSW, K4 KEYSW, K40 KEYSW, K41 KEYSW, K42 KEYSW, K43 KEYSW, K44 KEYSW, K45 KEYSW, K46 KEYSW, K47 KEYSW, K48 KEYSW, K49 KEYSW, K5 KEYSW, K50 KEYSW, K51 KEYSW, K52 KEYSW, K53 KEYSW, K54 KEYSW, K55 KEYSW, K56 KEYSW, K57 KEYSW, K58 KEYSW, K59 KEYSW, K6 KEYSW, K60 KEYSW, K7 KEYSW, K8 KEYSW, K9 KEYSW, U1 ARDUINO_PRO_MINI, U2 FT231X_breakout

Commit message: Keyboard layout done?
Parts:
- removed C1, C2, C3, C4: 0.1u, Capacitor_SMD:C_0805_2012Metric_Pad1.15x1.40mm_HandSolder, symbol Device:C
- removed C5: 4.7u, Capacitor_SMD:C_0805_2012Metric_Pad1.15x1.40mm_HandSolder, symbol Device:C
- removed JP1, JP2: JPR2, symbol Device:Jumper_NC_Small
- removed U1: ARDUINO_PRO_MINI, MODULE_ARDUINO_PRO_MINI, symbol ARDUINO_PRO_MINI:ARDUINO_PRO_MINI
- removed U2: FT231X_breakout, symbol tens:FT231X_breakout
- added C6: C, Diode_THT:D_DO-35_SOD27_P7.62mm_Horizontal, symbol Device:C
- added D61: LED, LED_THT:LED_D3.0mm, symbol Device:LED
- added H5, H6: MountingHole, MountingHole:MountingHole_3.2mm_M3_DIN965, symbol Mechanical:MountingHole
- added R1: 680, Resistor_THT:R_Axial_DIN0204_L3.6mm_D1.6mm_P7.62mm_Horizontal, symbol Device:R_US
- added R2: 10k, Resistor_THT:R_Axial_DIN0204_L3.6mm_D1.6mm_P7.62mm_Horizontal, symbol Device:R_US
- added U4: ATmega328P-PU, Package_DIP:DIP-28_W7.62mm, symbol MCU_Microchip_ATmega:ATmega328P-PU
- D0, D1, D10, D11, D12, D13, D14, D15, D16, D17, D18, D19, D2, D20, D21, D22, D23, D24, D25, D26, D27, D28, D29, D3, D30, D31, D32, D33, D34, D35, D36, D37, D38, D39, D4, D40, D41, D42, D43, D44, D45, D46, D47, D48, D49, D5, D50, D51, D52, D53, D54, D55, D56, D57, D58, D59, D6, D60, D7, D8, D9: footprint Diode_SMD:D_0805_2012Metric_Pad1.15x1.40mm_HandSolder -> Diode_THT:D_DO-35_SOD27_P7.62mm_Horizontal
- J1: footprint (none) -> Connector_PinSocket_2.54mm:PinSocket_2x03_P2.54mm_Vertical
- J2: footprint (none) -> Connector_PinSocket_2.54mm:PinSocket_1x06_P2.54mm_Vertical
Connections:
- net labels added: RxD, TxD
- net labels removed: RTS, RXI, TXO
- wire segments 177 -> 178
Other:
- note removed: "Bypass caps\nLEDs\nAux power\n"
- note removed: "FIGURE OUT RTS"
- note removed: "Install for programmming"
- moved on the sheet: J1, J2
