File: hardware/keyboard/minimal-60-v3/minimal-60-v3.kicad_pcb (KiCad board)
At the start: 2 copper layers, 143 parts, among them J1 USB_B_Micro, J2 Conn_02x03_Odd_Even, K0 KEYSW, K1 KEYSW, K10 KEYSW, K11 KEYSW, K12 KEYSW, K13 KEYSW, K14 KEYSW, K15 KEYSW, K16 KEYSW, K17 KEYSW, K18 KEYSW, K19 KEYSW, K2 KEYSW, K20 KEYSW, K21 KEYSW, K22 KEYSW, K23 KEYSW, K24 KEYSW, K25 KEYSW, K26 KEYSW, K27 KEYSW, K28 KEYSW, K29 KEYSW, K3 KEYSW, K30 KEYSW, K31 KEYSW, K32 KEYSW, K33 KEYSW, K34 KEYSW, K35 KEYSW, K36 KEYSW, K37 KEYSW, K38 KEYSW, K39 KEYSW, K4 KEYSW, K40 KEYSW, K41 KEYSW, K42 KEYSW, K43 KEYSW, K44 KEYSW, K45 KEYSW, K46 KEYSW, K47 KEYSW, K48 KEYSW, K49 KEYSW, K5 KEYSW, K50 KEYSW, K51 KEYSW, K52 KEYSW, K53 KEYSW, K54 KEYSW, K55 KEYSW, K56 KEYSW, K57 KEYSW, K58 KEYSW, K59 KEYSW, K6 KEYSW, K60 KEYSW, K7 KEYSW, K8 KEYSW, K9 KEYSW, SW1 Reset_SW, U1 ATmega32U4-AU, Y1 Crystal

Commit message: Keyboard layout done?
Parts:
- removed C1, C2, C3, C4: 0.1u, Capacitor_SMD:C_0805_2012Metric_Pad1.15x1.40mm_HandSolder
- removed C5: 4.7u, Capacitor_SMD:C_0805_2012Metric_Pad1.15x1.40mm_HandSolder
- removed C7: 22p, Capacitor_SMD:C_0805_2012Metric_Pad1.15x1.40mm_HandSolder
- removed C8: 1u, Capacitor_SMD:C_0805_2012Metric_Pad1.15x1.40mm_HandSolder
- removed R3: 22R, Resistor_SMD:R_0805_2012Metric_Pad1.15x1.40mm_HandSolder
- removed R4: 10k, Resistor_SMD:R_0805_2012Metric_Pad1.15x1.40mm_HandSolder
- removed SW1: Reset_SW, Button_Switch_SMD:SW_Push_1P1T_NO_6x6mm_H9.5mm
- removed U1: ATmega32U4-AU, Package_QFP:TQFP-44_10x10mm_P0.8mm
- removed Y1: Crystal, Crystal:Crystal_SMD_5032-2Pin_5.0x3.2mm_HandSoldering
- added D61: LED, LED_THT:LED_D3.0mm, F.Cu at (339.7, 59.7)
- added H5: MountingHole, MountingHole:MountingHole_3.2mm_M3_DIN965, F.Cu at (227.3, 59.7)
- added H6: MountingHole, MountingHole:MountingHole_3.2mm_M3_DIN965, F.Cu at (227.3, 161.3)
- added U4: ATmega328P-PU, Package_DIP:DIP-28_W7.62mm, B.Cu at (165.7, 146.1)
- C6: value 22p -> C; footprint Capacitor_SMD:C_0805_2012Metric_Pad1.15x1.40mm_HandSolder -> Capacitor_THT:C_Disc_D3.8mm_W2.6mm_P2.50mm
- D0, D1, D10, D11, D12, D13, D14, D15, D16, D17, D18, D19, D2, D20, D21, D22, D23, D24, D25, D26, D27, D28, D29, D3, D30, D31, D32, D33, D34, D35, D36, D37, D38, D39, D4, D40, D41, D42, D43, D44, D45, D46, D47, D48, D49, D50, D51, D52, D53, D54, D55, D56, D57, D58, D59, D6, D60, D7, D8, D9: footprint Diode_SMD:D_0805_2012Metric_Pad1.15x1.40mm_HandSolder -> Diode_THT:D_DO-35_SOD27_P7.62mm_Horizontal
- D5: footprint Diode_SMD:D_0805_2012Metric_Pad1.15x1.40mm_HandSolder -> Diode_THT:D_DO-35_SOD27_P7.62mm_Horizontal; moved to F.Cu
- J1: value USB_B_Micro -> Conn_02x03_Odd_Even; footprint Connector_USB:USB_Mini-B_Wuerth_65100516121_Horizontal -> Connector_PinSocket_2.54mm:PinSocket_2x03_P2.54mm_Vertical
- J2: value Conn_02x03_Odd_Even -> Conn_01x06; footprint Connector_PinHeader_2.54mm:PinHeader_2x03_P2.54mm_Vertical -> Connector_PinSocket_2.54mm:PinSocket_1x06_P2.54mm_Vertical
- R1: value 10k -> 680; footprint Resistor_SMD:R_0805_2012Metric_Pad1.15x1.40mm_HandSolder -> Resistor_THT:R_Axial_DIN0204_L3.6mm_D1.6mm_P7.62mm_Horizontal
- R2: value 22R -> 10k; footprint Resistor_SMD:R_0805_2012Metric_Pad1.15x1.40mm_HandSolder -> Resistor_THT:R_Axial_DIN0204_L3.6mm_D1.6mm_P7.62mm_Horizontal
- moved H2 208.3 mm to (69.8, 59.7)
- moved H4 205.9 mm to (69.8, 161.3)
- moved D56 196.4 mm to (221.6, 152.4)
- moved D53 195.2 mm to (94.0, 153.7)
- moved D0 183.7 mm to (78.7, 90.2)
- moved K0 182.4 mm to (87.3, 67.9)
- moved K1 182.4 mm to (106.4, 67.9)
- moved K11 182.4 mm to (296.9, 67.9)
- moved K12 182.4 mm to (315.9, 67.9)
- moved K13 182.4 mm to (344.5, 67.9)
- moved K14 182.4 mm to (92.1, 87.0)
- moved K15 182.4 mm to (115.9, 87.0)
- moved K17 182.4 mm to (154.0, 87.0)
- moved K18 182.4 mm to (173.1, 87.0)
- moved K2 182.4 mm to (125.4, 67.9)
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Connections:
- C6 pad 1: Net-(C6-Pad1) -> VCC
- D0 pad 1: /Row_0 -> /ROW0
- D1 pad 1: /Row_0 -> /ROW0
- D10 pad 1: /Row_0 -> /ROW5
- D11 pad 1: /Row_0 -> /ROW2
- D12 pad 1: /Row_0 -> /ROW0
- D13 pad 1: /Row_0 -> /ROW3
- D14 pad 1: /Row_1 -> /ROW1
- D15 pad 1: /Row_1 -> /ROW1
- D16 pad 1: /Row_1 -> /ROW4
- D17 pad 1: /Row_1 -> /ROW1
- D18 pad 1: /Row_1 -> /ROW5
- D19 pad 1: /Row_1 -> /ROW1
- D2 pad 1: /Row_0 -> /ROW3
- D20 pad 1: /Row_1 -> /ROW6
- D21 pad 1: /Row_1 -> /ROW1
- D22 pad 1: /Row_1 -> /ROW5
- D23 pad 1: /Row_1 -> /ROW1
- D24 pad 1: /Row_1 -> /ROW6
- D25 pad 1: /Row_1 -> /ROW3
- D26 pad 1: /Row_1 -> /ROW1
- D27 pad 1: /Row_1 -> /ROW4
- D28 pad 1: /Row_2 -> /ROW2
- D29 pad 1: /Row_2 -> /ROW2
- D3 pad 1: /Row_0 -> /ROW0
- D30 pad 1: /Row_2 -> /ROW5
- D31 pad 1: /Row_2 -> /ROW2
- D32 pad 1: /Row_2 -> /ROW6
- D33 pad 1: /Row_2 -> /ROW2
- D34 pad 1: /Row_2 -> /ROW7
- D35 pad 1: /Row_2 -> /ROW2
- D36 pad 1: /Row_2 -> /ROW6
- D37 pad 1: /Row_2 -> /ROW2
- D38 pad 1: /Row_2 -> /ROW7
- D39 pad 1: /Row_2 -> /ROW4
- D4 pad 1: /Row_0 -> /ROW4
- D40 pad 1: /Row_2 -> /ROW2
- D41 pad 1: /Row_3 -> /ROW3
- D42 pad 1: /Row_3 -> /ROW6
- D43 pad 1: /Row_3 -> /ROW6
- D44 pad 1: /Row_3 -> /ROW3
- D45 pad 1: /Row_3 -> /ROW7
- D46 pad 1: /Row_3 -> /ROW3
- D47 pad 1: /Row_3 -> /ROW7
- D48 pad 1: /Row_3 -> /ROW3
- D49 pad 1: /Row_3 -> /ROW7
- D5 pad 1: /Row_0 -> /ROW0
- D50 pad 1: /Row_3 -> /ROW3
- D51 pad 1: /Row_3 -> /ROW0
- D52 pad 1: /Row_3 -> /ROW5
- D53 pad 1: /Row_4 -> /ROW5
- D54 pad 1: /Row_4 -> /ROW4
- D55 pad 1: /Row_4 -> /ROW7
- D56 pad 1: /Row_4 -> /ROW4
- D57 pad 1: /Row_4 -> /ROW4
- D58 pad 1: /Row_4 -> Net-(D58-Pad1)
- D59 pad 1: /Row_4 -> /ROW6
- D6 pad 1: /Row_0 -> /ROW5
- D60 pad 1: /Row_4 -> /ROW7
- D7 pad 1: /Row_0 -> /ROW0
- D8 pad 1: /Row_0 -> /ROW4
- D9 pad 1: /Row_0 -> /ROW0
- J1 pad 1: VCC -> Net-(J1-Pad1)
- J1 pad 2: Net-(J1-Pad2) -> VCC
- J1 pad 5: GND -> Net-(J1-Pad5)
- J2 pad 1: VCC -> GND
- J2 pad 2: /Row_2 -> GND
- J2 pad 3: /Row_4 -> VCC
- J2 pad 4: /Row_3 -> /TxD
- J2 pad 5: GND -> /RxD
- J2 pad 6: /Reset -> Net-(J1-Pad5)
- K0 pad 1: /Col_0 -> /COL0
- K1 pad 1: /Col_1 -> /COL1
- K10 pad 1: /Col_10 -> /COL5
- K11 pad 1: /Col_11 -> /COL6
- K12 pad 1: /Col_12 -> /COL7
- K13 pad 1: /Col_13 -> /COL7
- K14 pad 1: /Col_0 -> /COL0
- K15 pad 1: /Col_1 -> /COL1
- K16 pad 1: /Col_2 -> /COL1
- K17 pad 1: /Col_3 -> /COL2
- K18 pad 1: /Col_4 -> /COL2
- K19 pad 1: /Col_5 -> /COL3
- K2 pad 1: /Col_2 -> /COL1
- K20 pad 1: /Col_6 -> /COL3
- K21 pad 1: /Col_7 -> /COL4
- K22 pad 1: /Col_8 -> /COL4
- K23 pad 1: /Col_9 -> /COL5
- K24 pad 1: /Col_10 -> /COL5
- K25 pad 1: /Col_11 -> /COL6
- K26 pad 1: /Col_12 -> /COL7
- K27 pad 1: /Col_13 -> /COL7
- K28 pad 1: /Col_0 -> /COL0
- K29 pad 1: /Col_1 -> /COL1
- K3 pad 1: /Col_3 -> /COL2
- K30 pad 1: /Col_2 -> /COL1
- K31 pad 1: /Col_3 -> /COL2
- K32 pad 1: /Col_4 -> /COL2
- K33 pad 1: /Col_5 -> /COL3
- K34 pad 1: /Col_6 -> /COL3
- K35 pad 1: /Col_7 -> /COL4
- K36 pad 1: /Col_8 -> /COL4
- K37 pad 1: /Col_9 -> /COL5
- K38 pad 1: /Col_10 -> /COL5
- K39 pad 1: /Col_11 -> /COL6
- K4 pad 1: /Col_4 -> /COL2
- K40 pad 1: /Col_12 -> /COL7
- K41 pad 1: /Col_0 -> /COL0
- K42 pad 1: /Col_1 -> /COL0
- K43 pad 1: /Col_2 -> /COL1
- K44 pad 1: /Col_3 -> /COL2
- K45 pad 1: /Col_4 -> /COL2
- K46 pad 1: /Col_5 -> /COL3
- K47 pad 1: /Col_6 -> /COL1
- K48 pad 1: /Col_7 -> /COL4
- K49 pad 1: /Col_8 -> /COL4
- K5 pad 1: /Col_5 -> /COL3
- K50 pad 1: /Col_9 -> /COL5
- K51 pad 1: /Col_10 -> /COL6
- K52 pad 1: /Col_11 -> /COL6
- K53 pad 1: /Col_0 -> /COL0
- K54 pad 1: /Col_1 -> /COL0
- K55 pad 1: /Col_2 -> /COL0
- K56 pad 1: /Col_3 -> /COL3
- K57 pad 1: /Col_4 -> /COL5
- K58 pad 1: /Col_5 -> /COL6
- K59 pad 1: /Col_6 -> /COL6
- K6 pad 1: /Col_6 -> /COL3
- K60 pad 1: /Col_7 -> /COL6
- K7 pad 1: /Col_7 -> /COL4
- K8 pad 1: /Col_8 -> /COL4
- K9 pad 1: /Col_9 -> /COL5
- R1 pad 1: /Reset -> Net-(R1-Pad1)
- R1 pad 2: VCC -> Net-(D61-Pad2)
- R2 pad 1: Net-(R2-Pad1) -> VCC
- R2 pad 2: Net-(J1-Pad3) -> Net-(J1-Pad5)
Routing:
- net /ROW4: track 0.00 -> 486.2 mm, vias 0 -> 8
- net /ROW5: track 0.00 -> 447.8 mm, vias 0 -> 6
- net /ROW3: track 0.00 -> 390.5 mm, vias 0 -> 5
- net /ROW6: track 0.00 -> 379.0 mm, vias 0 -> 5
- net /ROW0: track 0.00 -> 375.9 mm, vias 0 -> 2
- net /COL5: track 0.00 -> 340.0 mm, vias 0 -> 2
- net /ROW7: track 0.00 -> 333.9 mm, vias 0 -> 4
- net /ROW2: track 0.00 -> 322.6 mm, vias 0 -> 2
- net /COL6: track 0.00 -> 314.5 mm, vias 0 -> 3
- net /ROW1: track 0.00 -> 307.4 mm, vias 0 -> 1
- net /COL7: track 0.00 -> 293.7 mm, vias 0 -> 3
- net Net-(J1-Pad5): track 0.00 -> 273.1 mm, vias 0 -> 2
- net Net-(D61-Pad2): track 0.00 -> 260.8 mm, vias 0 -> 1
- net /TxD: track 0.00 -> 253.4 mm, vias 0 -> 2
- net /COL4: track 0.00 -> 249.6 mm, vias 0 -> 4
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- added copper zone on B.Cu, net GND
- added copper zone on F.Cu, net VCC
Other:
- board outline added: 302.3 x 109.2 mm
- net class Default: clearance 0.2 -> 0.1778; trace_width 0.25 -> 0.1778; via_dia 0.8 -> 0.508; via_drill 0.4 -> 0.254
- rule trace_clearance: 0.2 -> 0.1778
- rule trace_min: 0.2 -> 0.1778
- rule via_min_drill: 0.3 -> 0.254
- rule via_min_size: 0.4 -> 0.508

Commit message: more more cleaning
Other:
- board text added: "1"
- board text added: "E. Hazen -- 2021-11"
- board text added: "GND"
- board text added: "UPCO Graphics Systems -- Serial Keyboard -- Rev A"
