File: hardware/rc2014_vga/lcd_adapter.sch (KiCad schematic (older format))
At the start: 24 parts, among them J1 CMOD-A7, J2 Conn_01x02_Male, J3 Conn_02x14_Odd_Even, J4 DB15_Female, J5 Conn_01x33

Commit message: working on layout
Parts:
- removed J3: Conn_02x14_Odd_Even, Connector_PinHeader_2.54mm:PinHeader_2x14_P2.54mm_Vertical, symbol Connector_Generic:Conn_02x14_Odd_Even
- removed J?: Conn_01x06_Male, symbol Connector:Conn_01x06_Male
- removed U?: SN74LVCC4245A, symbol adapter_symbols:SN74LVCC4245A
- added C1, C2, C3, C4, C5, C7: 0.1uF, Capacitor_SMD:C_1206_3216Metric_Pad1.33x1.80mm_HandSolder, symbol Device:C_Small
- added C6, C8: 1uF, Capacitor_SMD:C_1206_3216Metric_Pad1.33x1.80mm_HandSolder, symbol Device:C_Small
- added J6: RC2014_BUS, myRC2014_footprints:RC2014_Header, symbol myRC2014:RC2014_BUS
- added JP2, JP3: Jumper_3_Bridged12, Connector_PinSocket_2.54mm:PinSocket_1x03_P2.54mm_Vertical, symbol Jumper:Jumper_3_Bridged12
- added U1, U2, U3, U4: SN74LV1T34DBV, Package_TO_SOT_SMD:SOT-23-5, symbol Logic_LevelTranslator:SN74LV1T34DBV
- added U5: LTC1844ES5-3.3, Package_TO_SOT_SMD:SOT-23-5_HandSoldering, symbol myRC2014:LTC1844ES5-3.3
- added X1: 100.00MHz, Package_TO_SOT_SMD:SOT-23-5_HandSoldering, symbol myRC2014:CXO_SOT23
- J7: renamed from J?; footprint (none) -> Connector_PinHeader_2.54mm:PinHeader_1x06_P2.54mm_Vertical
- J8: renamed from J?; footprint (none) -> Connector_PinSocket_2.54mm:PinSocket_2x03_P2.54mm_Vertical
- R1, R10, R11, R12, R13, R14, R2, R3, R4, R5, R6, R7, R8, R9: footprint Resistor_THT:R_Axial_DIN0414_L11.9mm_D4.5mm_P15.24mm_Horizontal -> Resistor_SMD:R_1206_3216Metric_Pad1.30x1.75mm_HandSolder
Connections:
- net labels added: KB_CLOCK, KB_DATA, RXA, RXB, TXA, TXB
- net labels removed: VGA_B0, VGA_B1, VGA_B2, VGA_B3, VGA_G0, VGA_G1, VGA_G2, VGA_G3, VGA_HS, VGA_R0, VGA_R1, VGA_R2, VGA_R3, VGA_VS
- wire segments 178 -> 200
Other:
- note removed: "CPU Interface"
- note removed: "Jumper all for VGA"
- moved on the sheet: J1, J7, J8

Commit message: Change all to TH
Parts:
- removed C7: 0.1uF, Capacitor_SMD:C_1206_3216Metric_Pad1.33x1.80mm_HandSolder, symbol Device:C_Small
- removed U1, U2, U3, U4: SN74LV1T34DBV, Package_TO_SOT_SMD:SOT-23-5, symbol Logic_LevelTranslator:SN74LV1T34DBV
- removed U5: LTC1844ES5-3.3, Package_TO_SOT_SMD:SOT-23-5_HandSoldering, symbol myRC2014:LTC1844ES5-3.3
- removed X1: 100.00MHz, Package_TO_SOT_SMD:SOT-23-5_HandSoldering, symbol myRC2014:CXO_SOT23
- added R15, R16, R18, R19, R22: 2k, Resistor_THT:R_Axial_DIN0204_L3.6mm_D1.6mm_P5.08mm_Horizontal, symbol Device:R_US
- added R17, R20, R21: 3k, Resistor_THT:R_Axial_DIN0204_L3.6mm_D1.6mm_P5.08mm_Horizontal, symbol Device:R_US
- added VR1: LM2937xT, Package_TO_SOT_THT:TO-220-3_Vertical, symbol Regulator_Linear:LM2937xT
- added X1: CXO_DIP8, Oscillator:Oscillator_DIP-8, symbol Oscillator:CXO_DIP8
- C1, C2, C3, C4, C5: footprint Capacitor_SMD:C_1206_3216Metric_Pad1.33x1.80mm_HandSolder -> Capacitor_THT:C_Disc_D5.0mm_W2.5mm_P2.50mm
- C6: value 1uF -> 0.1uF; footprint Capacitor_SMD:C_1206_3216Metric_Pad1.33x1.80mm_HandSolder -> Capacitor_THT:C_Disc_D5.0mm_W2.5mm_P2.50mm
- C8: value 1uF -> 10uF; footprint Capacitor_SMD:C_1206_3216Metric_Pad1.33x1.80mm_HandSolder -> Capacitor_THT:C_Disc_D5.0mm_W2.5mm_P2.50mm
- R1, R10, R11, R12, R13, R14, R2, R3, R4, R5, R6, R7, R8, R9: footprint Resistor_SMD:R_1206_3216Metric_Pad1.30x1.75mm_HandSolder -> Resistor_THT:R_Axial_DIN0204_L3.6mm_D1.6mm_P5.08mm_Horizontal
Connections:
- wire segments 200 -> 196
Other:
- note added: "Level shifter\n"bricolage""
- note added: "TODO:\n* Redo level shifters with 74HC\n* Change all to TH\n* 12V for backlight (dimmer)?\n"
- note removed: "TODO:\n* Power supplies: 3.3V (regulator)?\n* 12V for backlight (dimmer)?\n"
- moved on the sheet: JP1

Commit message: working on layout
Parts:
- removed J5: Conn_01x33, lcd_adapter:FH12-33S-0.5, symbol Connector_Generic:Conn_01x33
- added J3: Conn_01x34, Connector_PinHeader_2.54mm:PinHeader_2x17_P2.54mm_Vertical, symbol Connector_Generic:Conn_01x34
- R1, R10, R11, R12, R13, R14, R15, R16, R17, R18, R19, R2, R20, R21, R22, R3, R4, R5, R6, R7, R8, R9: footprint Resistor_THT:R_Axial_DIN0204_L3.6mm_D1.6mm_P5.08mm_Horizontal -> Resistor_THT:R_Axial_DIN0204_L3.6mm_D1.6mm_P2.54mm_Vertical
Other:
- note added: "LCD Panel\nNeed adapter to flex cable\nof same pinout"
- note removed: "LCD Panel"
