File: hardware/7220_mono/7220_mono.kicad_pcb (KiCad board)
At the start: 2 copper layers, 99.2 x 115 mm, 46 parts, among them J1 RC2014_BUS, J2 JUMPER, U1 UPD7220, U10 74LS373, U11 74LS74, U12 74S20, U13 74LS00, U14 74LS368, U15 CY62256-70PC, U16 CY62256-70PC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

Commit message: working on 7220
Parts:
- removed U14: 74LS368, Package_DIP:DIP-16_W7.62mm
- U15, U16: value CY62256-70PC -> CY7C199
- U20, U21: value 74S299 -> 74F299
- U3: value 74S37 -> 74AC04
- U5: value 74S04 -> 74AC04
- U7: value 74LS373 -> 74AC373
- X1: value CXO_DIP8 -> 40.000MHz
- moved U3 35.6 mm to (85.1, 123.2)
- moved U5 35.6 mm to (120.0, 123.2)
Connections:
- U11 pad 14: VCC -> (no net)
- U11 pad 7: GND -> (no net)
- U12 pad 14: VCC -> (no net)
- U12 pad 7: GND -> (no net)
- U2 pad 14: VCC -> (no net)
- U2 pad 7: GND -> (no net)
- U3 pad 1: Net-(U11-Pad9) -> Net-(U3-Pad1)
- U3 pad 10: Net-(U3-Pad10) -> /2xWCLK
- U3 pad 11: (no net) -> /~2xWCLK
- U3 pad 14: VCC -> (no net)
- U3 pad 2: Net-(U11-Pad9) -> /~PIX-CLK
- U3 pad 3: /VIDEO -> /~PIX-CLK
- U3 pad 4: /~PIX-CLK -> /PIX-CLK
- U3 pad 5: /~PIX-CLK -> /~DBIN
- U3 pad 6: /PIX-CLK -> /DBIN
- U3 pad 7: GND -> (no net)
- U3 pad 8: /~PIX-CLK -> /HSYNC
- U3 pad 9: Net-(U3-Pad10) -> Net-(U3-Pad9)
- U4 pad 14: VCC -> (no net)
- U4 pad 7: GND -> (no net)
- U5 pad 10: /VSR-LD -> /VSYNC
- U5 pad 11: Net-(U12-Pad6) -> Net-(U5-Pad11)
- U5 pad 14: VCC -> (no net)
- U5 pad 5: /~DBIN -> Net-(U11-Pad9)
- U5 pad 6: /DBIN -> /VIDEO
- U5 pad 7: GND -> (no net)
- U5 pad 8: /2xWCLK -> /VSR-LD
- U5 pad 9: /~2xWCLK -> Net-(U12-Pad6)
- U9 pad 3: Net-(U9-Pad3) -> Net-(U3-Pad9)
- U9 pad 6: Net-(U9-Pad6) -> Net-(U5-Pad11)
- X1 pad 5: Net-(U3-Pad10) -> Net-(U3-Pad1)
