File: hardware/7220_mono/7220_mono.sch (KiCad schematic (older format))
At the start: 41 parts, among them U1 UPD7220, U10 74LS373, U11 74LS74, U12 74S20, U14 74LS368, U15 CY62256-70PC, U16 CY62256-70PC, U2 74LS74, U20 74S299, U21 74S299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

Commit message: working on 7220
Parts:
- removed unit 3 of U11
- removed unit 3 of U12
- removed U14: 74LS368, Package_DIP:DIP-16_W7.62mm, symbol 74xx:74LS368
- removed unit 3 of U2
- removed U3: 74S37, Package_DIP:DIP-14_W7.62mm, symbol 74xx:74LS37
- removed unit 5 of U4
- removed U5: 74S04, Package_DIP:DIP-14_W7.62mm, symbol 74xx:74LS04
- added U3, U5: 74AC04, Package_DIP:DIP-14_W7.62mm, symbol 74xx:74HC04
- U12: CatNo (none) -> 296-34108-5-ND; Vendor (none) -> DigiKey
- U15, U16: value CY62256-70PC -> CY7C199; CatNo (none) -> 2156-CY7C199N-20PXC-ND; Vendor (none) -> DigiKey
- U20, U21: value 74S299 -> 74F299; CatNo (none) -> 4296-33908-5-ND; Vendor (none) -> DigiKey
- U4: CatNo (none) -> 296-1723-5-ND; Vendor (none) -> DigiKey
- U7: value 74LS373 -> 74AC373
- U8: CatNo (none) -> 296-3863-5-ND; Vendor (none) -> DigiKey
- X1: value CXO_DIP8 -> 40.000MHz; CatNo (none) -> X966-ND; Vendor (none) -> DigiKey
Connections:
- wire segments 346 -> 340
