File: hardware/7220_mono/cpu_if.sch (KiCad schematic (older format))
At the start: 5 parts, among them J1 RC2014_BUS, J2 JUMPER, U13 74LS00, U6 74LS682

Commit message: working on 7220
Parts:
- U6: CatNo (none) -> 296-14898-5-ND; Vendor (none) -> DigiKey
Changed lines of the file:
@@
 F 2 "Package_DIP:DIP-20_W7.62mm" H 5400 2200 50  0001 C CNN
 F 3 "" H 5400 2200 50  0001 C CNN
+F 4 "296-14898-5-ND" H 5400 2200 50  0001 C CNN "CatNo"
+F 5 "DigiKey" H 5400 2200 50  0001 C CNN "Vendor"
 	1    5400 2200
 	1    0    0    1

Commit message: Working on 2-board 7220
Parts:
- renumbered J1 to J?, J2 to J?, RN1 to RN?, U6 to U?, U13 to U?
Changed lines of the file:
@@
 $EndDescr
 $Comp
-L myRC2014:RC2014_BUS J1
+L myRC2014:RC2014_BUS J?
 U 1 1 61ECEBED
 P 2750 1400
-F 0 "J1" H 2558 1665 50  0000 C CNN
+F 0 "J?" H 2558 1665 50  0000 C CNN
 F 1 "RC2014_BUS" H 2558 1574 50  0000 C CNN
 F 2 "myRC2014_footprints:RC2014_Header" H 2750 1400 50  0001 C CNN
@@
 $EndComp
 $Comp
-L myRC2014:RC2014_BUS J1
+L myRC2014:RC2014_BUS J?
 U 2 1 61ECF849
 P 1400 3200
-F 0 "J1" H 1158 3465 50  0000 C CNN
+F 0 "J?" H 1158 3465 50  0000 C CNN
 F 1 "RC2014_BUS" H 1158 3374 50  0000 C CNN
 F 2 "myRC2014_footprints:RC2014_Header" H 1400 3200 50  0001 C CNN
@@
 $EndComp
 $Comp
-L 74xx_IEEE:74LS682 U6
+L 74xx_IEEE:74LS682 U?
 U 1 1 61ED7678
 P 5400 2200
-F 0 "U6" H 5400 1134 50  0000 C CNN
+F 0 "U?" H 5400 1134 50  0000 C CNN
 F 1 "74LS682" H 5400 1225 50  0000 C CNN
 F 2 "Package_DIP:DIP-20_W7.62mm" H 5400 2200 50  0001 C CNN
@@
 	3100 5200 2750 5200
 $Comp
-L 74xx:74LS00 U13
+L 74xx:74LS00 U?
 U 1 1 61EF5496
 P 6450 4350
-F 0 "U13" H 6450 4675 50  0000 C CNN
+F 0 "U?" H 6450 4675 50  0000 C CNN
 F 1 "74LS00" H 6450 4584 50  0000 C CNN
 F 2 "Package_DIP:DIP-14_W7.62mm" H 6450 4350 50  0001 C CNN
@@
 	5950 4250 6150 4250
 $Comp
-L 74xx:74LS00 U13
+L 74xx:74LS00 U?
 U 2 1 61EFEA33
 P 6450 5050
-F 0 "U13" H 6450 5375 50  0000 C CNN
+F 0 "U?" H 6450 5375 50  0000 C CNN
 F 1 "74LS00" H 6450 5284 50  0000 C CNN
 F 2 "Package_DIP:DIP-14_W7.62mm" H 6450 5050 50  0001 C CNN
@@
 A0
 $Comp
-L power:GND #PWR047
+L power:GND #PWR?
 U 1 1 61F04705
 P 2900 3200
-F 0 "#PWR047" H 2900 2950 50  0001 C CNN
+F 0 "#PWR?" H 2900 2950 50  0001 C CNN
 F 1 "GND" H 2900 3250 50  0000 C CNN
 F 2 "" H 2900 3200 50  0001 C CNN
@@
 	3150 3000 2750 3000
 $Comp
-L power:VCC #PWR048
+L power:VCC #PWR?
 U 1 1 61F077A7
 P 3050 3300
-F 0 "#PWR048" H 3050 3150 50  0001 C CNN
+F 0 "#PWR?" H 3050 3150 50  0001 C CNN
 F 1 "VCC" H 3065 3473 50  0000 C CNN
 F 2 "" H 3050 3300 50  0001 C CNN
@@
 	3050 3400 2750 3400
 $Comp
-L power:GND #PWR045
+L power:GND #PWR?
 U 1 1 61F0B47C
 P 1600 3200
-F 0 "#PWR045" H 1600 2950 50  0001 C CNN
+F 0 "#PWR?" H 1600 2950 50  0001 C CNN
 F 1 "GND" H 1600 3250 50  0000 C CNN
 F 2 "" H 1600 3200 50  0001 C CNN
@@
 	1800 3400 1800 3350
 $Comp
-L power:VCC #PWR046
+L power:VCC #PWR?
 U 1 1 61F0D1E8
 P 1800 3350
-F 0 "#PWR046" H 1800 3200 50  0001 C CNN
+F 0 "#PWR?" H 1800 3200 50  0001 C CNN
 F 1 "VCC" H 1815 3523 50  0000 C CNN
 F 2 "" H 1800 3350 50  0001 C CNN
@@
 $EndComp
 $Comp
-L 74xx:74LS00 U13
+L 74xx:74LS00 U?
 U 5 1 61F0D53B
 P 6450 6050
-F 0 "U13" H 6400 6100 50  0000 L CNN
+F 0 "U?" H 6400 6100 50  0000 L CNN
 F 1 "74LS00" H 6350 6000 50  0000 L CNN
 F 2 "Package_DIP:DIP-14_W7.62mm" H 6450 6050 50  0001 C CNN
@@
 $EndComp
 $Comp
-L power:VCC #PWR053
+L power:VCC #PWR?
 U 1 1 61F0FB3F
 P 6450 5550
-F 0 "#PWR053" H 6450 5400 50  0001 C CNN
+F 0 "#PWR?" H 6450 5400 50  0001 C CNN
 F 1 "VCC" H 6465 5723 50  0000 C CNN
 F 2 "" H 6450 5550 50  0001 C CNN
@@
 $EndComp
 $Comp
-L power:GND #PWR054
+L power:GND #PWR?
 U 1 1 61F101E3
 P 6450 6550
-F 0 "#PWR054" H 6450 6300 50  0001 C CNN
+F 0 "#PWR?" H 6450 6300 50  0001 C CNN
 F 1 "GND" H 6450 6400 50  0000 C CNN
 F 2 "" H 6450 6550 50  0001 C CNN
@@
 $EndComp
 $Comp
-L Connector_Generic:Conn_02x06_Odd_Even J2
+L Connector_Generic:Conn_02x06_Odd_Even J?
 U 1 1 61F119A5
 P 3500 1600
-F 0 "J2" H 3550 2017 50  0000 C CNN
+F 0 "J?" H 3550 2017 50  0000 C CNN
 F 1 "JUMPER" H 3550 1926 50  0000 C CNN
 F 2 "Connector_PinHeader_2.54mm:PinHeader_2x06_P2.54mm_Vertical" H 3500 1600 50  0001 C CNN
@@
 	3800 1900 4550 1900
 $Comp
-L power:VCC #PWR051
+L power:VCC #PWR?
 U 1 1 61F2B71E
 P 4350 2150
-F 0 "#PWR051" H 4350 2000 50  0001 C CNN
+F 0 "#PWR?" H 4350 2000 50  0001 C CNN
 F 1 "VCC" H 4365 2323 50  0000 C CNN
 F 2 "" H 4350 2150 50  0001 C CNN
@@
 	4500 2000 4850 2000
 $Comp
-L power:GND #PWR052
+L power:GND #PWR?
 U 1 1 61F2CDD5
 P 4700 2100
-F 0 "#PWR052" H 4700 1850 50  0001 C CNN
+F 0 "#PWR?" H 4700 1850 50  0001 C CNN
 F 1 "GND" H 4700 2150 50  0000 C CNN
 F 2 "" H 4700 2100 50  0001 C CNN
@@
 	4700 2100 4850 2100
 $Comp
-L Device:R_Network06 RN1
+L Device:R_Network06 RN?
 U 1 1 61F2EAA4
 P 4350 1050
-F 0 "RN1" H 4638 1096 50  0000 L CNN
+F 0 "RN?" H 4638 1096 50  0000 L CNN
 F 1 "10k" H 4638 1005 50  0000 L CNN
 F 2 "Resistor_THT:R_Array_SIP7" V 4725 1050 50  0001 C CNN
@@
 	4550 1900 4850 1900
 $Comp
-L power:VCC #PWR050
+L power:VCC #PWR?
 U 1 1 61F37FA1
 P 4050 750
-F 0 "#PWR050" H 4050 600 50  0001 C CNN
+F 0 "#PWR?" H 4050 600 50  0001 C CNN
 F 1 "VCC" H 4065 923 50  0000 C CNN
 F 2 "" H 4050 750 50  0001 C CNN
@@
 	3300 1800 3300 1900
 $Comp
-L power:GND #PWR049
+L power:GND #PWR?
 U 1 1 61F3B3C3
 P 3300 2050
-F 0 "#PWR049" H 3300 1800 50  0001 C CNN
+F 0 "#PWR?" H 3300 1800 50  0001 C CNN
 F 1 "GND" H 3450 2000 50  0000 C CNN
 F 2 "" H 3300 2050 50  0001 C CNN
