File: hardware/eeprom-mega/KiCAD/eeprom-shield/eeprom-shield.kicad_pcb (KiCad board)
At the start: 2 copper layers, 101.6 x 53.3 mm, 21 parts, among them J1 Power, J2 PWM, J3 Analog, J4 PWM, J5 Analog, J6 Communication, J7 Digital, SW1 SW_SPST, U1 28C256

Commit message: EEPROM shield as built, arduino code to drive
Parts:
- removed SW1: SW_SPST, Connector_PinHeader_2.54mm:PinHeader_1x02_P2.54mm_Vertical
- added SW2: SW_SPDT, my_slide_sw:sw_spdt_2.54mm, F.Cu at (147.0, 92.4)
- added SW3: SW_SPDT, my_slide_sw:sw_spdt_2.54mm, F.Cu at (108.3, 55.0)
- U1: footprint Package_DIP:DIP-28_W15.24mm_Socket_LongPads -> my_zif_28:DIP_Socket-28_W11.9_W12.7_W15.24_W17.78_W18.5_3M_228-1277-00-0602J
Connections:
- J7 pad 11: /*44 -> /44
- J7 pad 12: /*45 -> /45
- J7 pad 9: /*46 -> /46
- U1 pad 28: +5V -> Net-(SW3-A)
Routing:
- net Net-(SW3-A): track 0.00 -> 13.5 mm
- net /27: track 84.0 -> 86.0 mm
- net Net-(SW2-A): track 64.8 -> 65.9 mm
Other:
- board text added: "->PWR ON"
- board text added: "1"
- board text added: "5V Only"
- board text added: "<-WR ENA"
- board text removed: "WR ENA"
