File: hardware/z180_test/z180_test.kicad_sch (KiCad schematic)
At the start: 18 parts, among them J1 Conn_01x06, J2 Conn_01x06, U1 Z180, U2 28C256, U3 AS6C4008-55PCN, X1 OSC 12.288MHz 5V

Commit message: working on z180 sch
Parts:
- added J3: DIN41612_02x32_AB, symbol Connector:DIN41612_02x32_AB
- added R11: R_US, symbol Device:R_US
- added U4, U8: 74LS139, symbol 74xx:74LS139
- added U5: 74LS245, symbol 74xx:74LS245
- added U6, U7, U9: 74LS244, symbol 74xx:74LS244
Connections:
- net GND: now also U1.1 (VSS), U1.18 (VSS), U1.2 (VSS), U1.36 (VSS), U2.27 (~{WE}), U5.10 (GND), U6.1 (OEa), U6.10 (GND), U6.19 (OEb), U7.1 (OEa), U7.10 (GND), U7.19 (OEb)
- net VCC: now also U1.10 (nINT0), U1.11 (nINT1), U1.12 (nINT2), U1.34 (VDD), U1.5 (nWAIT), U1.58 (nDREQ1), U1.7 (nBUSREQ), U1.9 (nNMI), R11.1
- net A0: now reaches U1.14 (A0)
- net A0: now also U2.10 (A0), U3.12 (A0), U7.17 (I3b)
- net A1: now reaches U1.15 (A1)
- net A1: now also U2.9 (A1), U3.11 (A1), U7.15 (I2b)
- net A2: now reaches U1.16 (A2)
- net A2: now also U2.8 (A2), U3.10 (A2), U7.13 (I1b)
- net A3: now reaches U1.17 (A3)
- net A3: now also U2.7 (A3), U3.9 (A3), U7.11 (I0b)
- net A4: now reaches U1.19 (A4)
- net A4: now also U2.6 (A4), U3.8 (A4), U7.8 (I3a)
- net A5: now reaches U1.20 (A5)
- net A5: now also U2.5 (A5), U3.7 (A5), U7.6 (I2a)
- net A6: now reaches U1.21 (A6)
- net A6: now also U2.4 (A6), U3.6 (A6), U7.4 (I1a)
- net A7: now reaches U1.22 (A7)
- net A7: now also U2.3 (A7), U3.5 (A7), U7.2 (I0a)
- net A8: now reaches U1.23 (A8)
- net A8: now also U2.25 (A8), U3.27 (A8), U6.17 (I3b)
- net A9: now reaches U1.24 (A9)
- net A9: now also U2.24 (A9), U3.26 (A9), U6.15 (I2b)
- net A10: now reaches U1.25 (A10)
- net A10: now also U2.21 (A10), U3.23 (A10), U6.13 (I1b)
- net A11: now reaches U1.26 (A11)
- net A11: now also U2.23 (A11), U3.25 (A11), U6.11 (I0b)
- net A12: now reaches U1.27 (A12)
- net A12: now also U2.2 (A12), U3.4 (A12), U6.8 (I3a)
- net A13: now reaches U1.28 (A13)
- net A13: now also U2.26 (A13), U3.28 (A13), U6.6 (I2a)
- net A14: now reaches U1.29 (A14)
- net A14: now also U2.1 (A14), U3.3 (A14), U6.4 (I1a)
- net A15: now reaches U1.30 (A15)
- net A15: now also U3.31 (A15), U6.2 (I0a)
- net A16: now reaches U1.31 (A16)
- net A16: now also U3.2 (A16), U9.8 (I3a)
- net A17: now reaches U1.32 (A17)
- net A17: now also U3.30 (A17), U8.14 (A0), U9.6 (I2a)
- net A18: now reaches U1.33 (A18_Tout)
- net A18: now also U3.1 (A18), U8.13 (A1), U9.4 (I1a)
- net A19: now reaches U1.35 (A19)
- net A19: now also U4.2 (A0), U9.2 (I0a)
- net D0: now reaches U1.37 (D0)
- net D0: now also U2.11 (D0), U3.13 (DQ0), U5.11 (B7)
- net D1: now reaches U1.38 (D1)
- net D1: now also U2.12 (D1), U3.14 (DQ1), U5.12 (B6)
- net D2: now reaches U1.39 (D2)
- net D2: now also U2.13 (D2), U3.15 (DQ2), U5.13 (B5)
- net D3: now reaches U1.40 (D3)
- net D3: now also U2.15 (D3), U3.17 (DQ3), U5.14 (B4)
- net D4: now reaches U1.41 (D4)
- net D4: now also U2.16 (D4), U3.18 (DQ4), U5.15 (B3)
- net D5: now reaches U1.42 (D5)
- net D5: now also U2.17 (D5), U3.19 (DQ5), U5.16 (B2)
- net D6: now reaches U1.43 (D6)
- net D6: now also U2.18 (D6), U3.20 (DQ6), U5.17 (B1)
- net D7: now reaches U1.44 (D7)
- net D7: now also U2.19 (D7), U3.21 (DQ7), U5.18 (B0)
- net nIORQ: now reaches U1.62 (nIORQ)
- net nIORQ: now also U9.13 (I1b)
- net nMREQ: now reaches U1.63 (nMREQ)
- net nMREQ: now also U4.1 (E), U9.11 (I0b)
- net nWR: now reaches U1.66 (nWR)
- net nWR: now also U3.29 (WE#), U9.17 (I3b)
- net nRD: now reaches U1.67 (nRD)
- net nRD: now also U3.24 (OE#), U5.1 (A->B), U9.15 (I2b)
- net at U1.8 (nRESET): now also R11.2
- net nROM: now reaches U2.20 (~{CS})
- net nROM: now also U8.12 (O0)
- net nRAM: now reaches U3.22 (CE#)
- net nRAM: now also U4.5 (O1)
- new net: U4.4 (O0), U8.15 (E)
- new net BA0: J3.a1 (Pin_a1), U7.3 (O3b)
- new net BA1: J3.a2 (Pin_a2), U7.5 (O2b)
- new net BA10: J3.a11 (Pin_a11), U6.7 (O1b)
- new net BA11: J3.a12 (Pin_a12), U6.9 (O0b)
- new net BA12: J3.a13 (Pin_a13), U6.12 (O3a)
- new net BA13: J3.a14 (Pin_a14), U6.14 (O2a)
- new net BA14: J3.a15 (Pin_a15), U6.16 (O1a)
- new net BA15: J3.a16 (Pin_a16), U6.18 (O0a)
- new net BA16: J3.a17 (Pin_a17), U9.12 (O3a)
- new net BA17: J3.a18 (Pin_a18), U9.14 (O2a)
- new net BA18: J3.a19 (Pin_a19), U9.16 (O1a)
- new net BA19: J3.a20 (Pin_a20), U9.18 (O0a)
- new net BA2: J3.a3 (Pin_a3), U7.7 (O1b)
- new net BA3: J3.a4 (Pin_a4), U7.9 (O0b)
- new net BA4: J3.a5 (Pin_a5), U7.12 (O3a)
- new net BA5: J3.a6 (Pin_a6), U7.14 (O2a)
- new net BA6: J3.a7 (Pin_a7), U7.16 (O1a)
- new net BA7: J3.a8 (Pin_a8), U7.18 (O0a)
- new net BA8: J3.a9 (Pin_a9), U6.3 (O3b)
- new net BA9: J3.a10 (Pin_a10), U6.5 (O2b)
- new net BD0: J3.a25 (Pin_a25), U5.9 (A7)
- new net BD1: J3.a26 (Pin_a26), U5.8 (A6)
- new net BD2: J3.a27 (Pin_a27), U5.7 (A5)
- new net BD3: J3.a28 (Pin_a28), U5.6 (A4)
- new net BD4: J3.a29 (Pin_a29), U5.5 (A3)
- new net BD5: J3.a30 (Pin_a30), U5.4 (A2)
- new net BD6: J3.a31 (Pin_a31), U5.3 (A1)
- new net BD7: J3.a32 (Pin_a32), U5.2 (A0)
- new net BIORQ: J3.a22 (Pin_a22), U9.7 (O1b)
- new net BMREQ: J3.a21 (Pin_a21), U9.9 (O0b)
- new net BRD: J3.a23 (Pin_a23), U9.5 (O2b)
- new net BWR: J3.a24 (Pin_a24), U9.3 (O3b)
- new net nEX1: U8.11 (O1)
- new net nEX2: U8.10 (O2)
- new net nEX3: U8.9 (O3)
- new net nEXTIO: U5.19 (CE)
- no-connect marks 1 -> 7
Other:
- moved on the sheet: C1, J1, J2, JP1, R1, R10, R2, R3, R4, R5, R6, R7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

Commit message: schem work
Parts:
- added D1: LED, symbol Device:LED
- added R12: 1k, symbol Device:R_US
- added U10, U7: 74AHC32, symbol 74xx:74LS32
- renumbered J3 to J1, J1 to J2, J2 to J3, R11 to R1, R6 to R11, R1 to R2, R2 to R3, R3 to R4, R4 to R5, R5 to R6, R8 to R7, R9 to R8, R7 to R9, U9 to U1, U6 to U2, U7 to U3, U5 to U4, U1 to U5, U8 to U6, U4 to U6, U2 to U8, U3 to U9
Connections:
- net A16: now also U6.14 (A0)
- net A17: no longer U6.14 (A0)
- net A18: now also U6.2 (A0); no longer U6.13 (A1)
- net A19: now also U6.3 (A1); no longer U6.2 (A0)
- net GND: now also J1.b10 (Pin_b10), J1.b11 (Pin_b11), J1.b12 (Pin_b12), J1.b13 (Pin_b13), J1.b14 (Pin_b14), J1.b15 (Pin_b15), J1.b16 (Pin_b16), J1.b25 (Pin_b25), J1.b26 (Pin_b26), J1.b27 (Pin_b27), J1.b28 (Pin_b28), J1.b29 (Pin_b29), J1.b30 (Pin_b30), J1.b31 (Pin_b31), J1.b32 (Pin_b32), J1.b5 (Pin_b5), J1.b6 (Pin_b6), J1.b7 (Pin_b7), J1.b8 (Pin_b8), J1.b9 (Pin_b9), U1.10 (GND), U6.13 (A1), U10.10, U7.10
- net VCC: now also J1.b1 (Pin_b1), J1.b2 (Pin_b2), J1.b3 (Pin_b3), J1.b4 (Pin_b4), U1.20 (VCC), U2.20 (VCC), U3.20 (VCC), U4.20 (VCC), R12.1
- net nIORQ: now also U6.15 (E)
- net nRAM: now also U7.3; no longer U6.5 (O1)
- net nRD: now also U8.22 (~{OE})
- net nROM: now also U6.4 (O0); no longer U6.12 (O0)
- net at U5.60 (nHALT): now also D1.1 (K)
- net M1: now reaches U5.65 (nM1)
- net CLK: now reaches U5.68 (PHI)
- net CLK: now also U10.9
- net at U6.6 (O2): now also U7.1
- net at U6.7 (O3): now also U7.2
- net BM1: now reaches J1.b22 (Pin_b22)
- net BM1: now also U7.8
- net BCLK: now reaches J1.b23 (Pin_b23)
- net BCLK: now also U10.8
- net nEX1: no longer names the net of U6.11 (O1)
- net nEX1: now also U7.5
- net nEX2: no longer names the net of U6.10 (O2)
- net nEX3: no longer names the net of U6.9 (O3)
- net nEXTIO renamed nDBUF
- net nDBUF: now also U7.6
- new net: D1.2 (A), R12.2
- new net nM1: U7.9
- new net nXMEM: U6.5 (O1), U7.4
- no-connect marks 7 -> 6
Other:
- note added: "Data buffer enable"
- note added: "Decode IO: 0000 - 00FF = on-board I/O 8000 - 80FF = off-board I/O (Incompletely decoded)"
- note added: "Decode MEM: 0.0000 - 3.FFFF = ROM (32k dup) 4.0000 - 7.FFFF = External mem (256k) 8.0000 - F.FFFF = RAM (512k)"
- note added: "Expansion Bus"
- moved on the sheet: U4, U6A, U6B

Commit message: schematic ~ done
Parts:
- added C1, C10, C11, C2, C3, C4, C6, C7, C9: .01uF, Capacitor_THT:C_Disc_D5.0mm_W2.5mm_P2.50mm, symbol Device:C_Small
- added C8: 1uF, Capacitor_THT:C_Disc_D5.0mm_W2.5mm_P2.50mm, symbol Device:C_Small
- added D2: LED, LED_THT:LED_D3.0mm, symbol Device:LED
- added D3: D, Diode_THT:D_T-1_P10.16mm_Horizontal, symbol Device:D
- added J1, J3: Conn_01x04, Connector_PinHeader_2.54mm:PinHeader_1x04_P2.54mm_Vertical, symbol Connector_Generic:Conn_01x04
- added J6: Conn_02x17_Counter_Clockwise, Connector_PinHeader_2.54mm:PinHeader_2x17_P2.54mm_Vertical, symbol Connector_Generic:Conn_02x17_Counter_Clockwise
- added R2: 1k, Resistor_THT:R_Axial_DIN0207_L6.3mm_D2.5mm_P10.16mm_Horizontal, symbol Device:R_US
- added SW1: SW_Push, Button_Switch_Keyboard:SW_Cherry_MX_1.00u_PCB, symbol Switch:SW_Push
- added unit 5 of U1
- added U10: 8255A, Package_DIP:DIP-40_W15.24mm, symbol Interface:8255A
- added U7: 74HC04, Package_DIP:DIP-14_W7.62mm, symbol 74xx:74HC04
- added unit 3 of U8
- added U9: 74HC14, Package_DIP:DIP-14_W7.62mm, symbol 74xx:74HC14
- C5: renamed from C1; value C_Small -> .01uF; footprint (none) -> Capacitor_THT:C_Disc_D5.0mm_W2.5mm_P2.50mm
- D1: footprint (none) -> LED_THT:LED_D3.0mm
- J2: renamed from J1; footprint (none) -> Connector_DIN:DIN41612_B_2x32_Female_Vertical_THT
- J4: renamed from J2; footprint (none) -> Connector_PinHeader_2.54mm:PinHeader_1x06_P2.54mm_Vertical
- J5: renamed from J3; footprint (none) -> Connector_PinHeader_2.54mm:PinHeader_1x06_P2.54mm_Vertical
- JP1: footprint (none) -> Connector_PinHeader_2.54mm:PinHeader_1x02_P2.54mm_Vertical
- R1: renamed from R12; footprint (none) -> Resistor_THT:R_Axial_DIN0207_L6.3mm_D2.5mm_P10.16mm_Horizontal
- R10: renamed from R1; value R_US -> 100k; footprint (none) -> Resistor_THT:R_Axial_DIN0207_L6.3mm_D2.5mm_P10.16mm_Horizontal
- R11: renamed from R9; footprint (none) -> Resistor_THT:R_Axial_DIN0207_L6.3mm_D2.5mm_P10.16mm_Horizontal
- R12: renamed from R10; footprint (none) -> Resistor_THT:R_Axial_DIN0207_L6.3mm_D2.5mm_P10.16mm_Horizontal
- R13: renamed from R11; footprint (none) -> Resistor_THT:R_Axial_DIN0207_L6.3mm_D2.5mm_P10.16mm_Horizontal
- R3: renamed from R2; footprint (none) -> Resistor_THT:R_Axial_DIN0207_L6.3mm_D2.5mm_P10.16mm_Horizontal
- R4: renamed from R3; footprint (none) -> Resistor_THT:R_Axial_DIN0207_L6.3mm_D2.5mm_P10.16mm_Horizontal
- R5: renamed from R4; footprint (none) -> Resistor_THT:R_Axial_DIN0207_L6.3mm_D2.5mm_P10.16mm_Horizontal
- R6: renamed from R5; footprint (none) -> Resistor_THT:R_Axial_DIN0207_L6.3mm_D2.5mm_P10.16mm_Horizontal
- R7: renamed from R6; footprint (none) -> Resistor_THT:R_Axial_DIN0207_L6.3mm_D2.5mm_P10.16mm_Horizontal
- R8: renamed from R7; footprint (none) -> Resistor_THT:R_Axial_DIN0207_L6.3mm_D2.5mm_P10.16mm_Horizontal
- R9: renamed from R8; footprint (none) -> Resistor_THT:R_Axial_DIN0207_L6.3mm_D2.5mm_P10.16mm_Horizontal
- U1: renamed from U10; footprint (none) -> Package_DIP:DIP-14_W7.62mm
- U1: renamed from U7; footprint (none) -> Package_DIP:DIP-14_W7.62mm
- U11: renamed from U8; footprint (none) -> Package_DIP:DIP-28_W15.24mm
- U2: renamed from U1; footprint (none) -> Package_DIP:DIP-20_W7.62mm
- U3: renamed from U2; footprint (none) -> Package_DIP:DIP-20_W7.62mm
- U4: renamed from U3; footprint (none) -> Package_DIP:DIP-20_W7.62mm
- U5: renamed from U4; footprint (none) -> Package_DIP:DIP-20_W7.62mm
- U8: renamed from U6; footprint (none) -> Package_DIP:DIP-16_W7.62mm
- renumbered U9 to U12, U5 to U6
Connections:
- net A0: now also U10.8 (A1)
- net A1: now also U10.9 (A0)
- net A17: now also U8.13 (A1)
- net BCLK: now also U1.11; no longer U1.8
- net CLK: now also U1.12; no longer U1.9
- net D0: now also U10.27 (D7)
- net D1: now also U10.28 (D6)
- net D2: now also U10.29 (D5)
- net D3: now also U10.30 (D4)
- net D4: now also U10.31 (D3)
- net D5: now also U10.32 (D2)
- net D6: now also U10.33 (D1)
- net D7: now also U10.34 (D0)
- net GND: now also U1.13, U6.50 (CKA0/DREQ0), C1.2, C10.2, C11.2, C2.2, C3.2, C4.2, C6.2, C7.2, C8.2, C9.2, J1.3 (Pin_3), J1.4 (Pin_4), J3.4 (Pin_4), J6.18 (Pin_18), J6.19 (Pin_19), J6.20 (Pin_20), J6.21 (Pin_21), J6.22 (Pin_22), J6.23 (Pin_23), SW1.2, U1.7 (GND), U10.7 (GND), U7.7 (GND), U8.8 (GND); no longer U1.10, U8.13 (A1)
- net VCC: now also U11.28 (VCC), U12.32 (VCC), C1.1, C10.1, C11.1, C2.1, C3.1, C4.1, C6.1, C7.1, C9.1, D3.1 (K), J1.1 (Pin_1), J1.2 (Pin_2), R2.1, U1.14 (VCC), U10.26 (VCC), U7.14 (VCC), U8.16 (VCC)
- net nRD: now also U10.5 (~{RD})
- net nWR: now also U10.36 (~{WR})
- net at R6.1, U6.45 (nRTS0): now also D2.1 (K)
- net at U6.55 (TXS): now also J3.1 (Pin_1)
- net at U6.56 (RXS/CTS1): now also J3.2 (Pin_2)
- net at U6.57 (CKS): now also J3.3 (Pin_3)
- net at R10.2: now also C8.1, D3.2 (A), SW1.1, U9.5; no longer U6.8 (nRESET)
- net nGPIO: now reaches U8.10 (O2)
- net nGPIO: now also U10.6 (~{CS})
- new net: U9.3, U9.6
- new net: J6.1 (Pin_1), U10.4 (PA0)
- new net: J6.10 (Pin_10), U10.18 (PB0)
- new net: J6.11 (Pin_11), U10.19 (PB1)
- new net: J6.12 (Pin_12), U10.20 (PB2)
- new net: J6.13 (Pin_13), U10.21 (PB3)
- new net: J6.14 (Pin_14), U10.22 (PB4)
- new net: J6.15 (Pin_15), U10.23 (PB5)
- new net: J6.16 (Pin_16), U10.24 (PB6)
- new net: J6.17 (Pin_17), U10.25 (PB7)
- new net: J6.2 (Pin_2), U10.3 (PA1)
- new net: J6.3 (Pin_3), U10.2 (PA2)
- new net: J6.4 (Pin_4), U10.1 (PA3)
- new net: J6.5 (Pin_5), U10.40 (PA4)
- new net: J6.6 (Pin_6), U10.39 (PA5)
- new net: J6.7 (Pin_7), U10.38 (PA6)
- new net: J6.8 (Pin_8), U10.37 (PA7)
- new net: D2.2 (A), R2.2
- new net PC0: J6.34 (Pin_34), U10.14 (PC0)
- new net PC1: J6.33 (Pin_33), U10.15 (PC1)
- new net PC2: J6.32 (Pin_32), U10.16 (PC2)
- new net PC3: J6.31 (Pin_31), U10.17 (PC3)
- new net PC4: J6.30 (Pin_30), U10.13 (PC4)
- new net PC5: J6.29 (Pin_29), U10.12 (PC5)
- new net PC6: J6.28 (Pin_28), U10.11 (PC6)
- new net PC7: J6.27 (Pin_27), U10.10 (PC7)
- new net RESET: U10.35 (RESET), U7.2
- new net nRESET: U6.8 (nRESET), U7.1, U9.4
- no-connect marks 6 -> 7
Other:
- note added: "Decode IO: 0000 - 00FF = on-board I/O 1000 - 10FF = off-board I/O 2000 - 20FF = 8255 3000 - 30FF = spare (Incompletely decoded)"
- note added: "POWER"
- note removed: "Decode IO: 0000 - 00FF = on-board I/O 8000 - 80FF = off-board I/O (Incompletely decoded)"
- moved on the sheet: R10, U11, U12

Commit message: tentative placement
Parts:
- removed X1: OSC 12.288MHz 5V, Oscillator:Oscillator_SeikoEpson_SG-8002DC, symbol Oscillator:SG-8002DC
- added C12, C13, C14: .01uF, Capacitor_THT:C_Disc_D5.0mm_W2.5mm_P2.50mm, symbol Device:C_Small
- added X1: ACO-xxxMHz-A, Oscillator:Oscillator_DIP-14, symbol Oscillator:ACO-xxxMHz-A
Connections:
- net GND: now also C12.2, C13.2, C14.2, X1.7 (GND)
- net VCC: now also C12.1, C13.1, C14.1, X1.14 (Vcc)
- net at R3.2, U6.4 (EXTAL): now also X1.8 (OUT)

Commit message: placement
Parts:
- added H1, H2, H3, H4, H5, H6, H7, H8: MountingHole, MountingHolesInch:Mtg4-40, symbol Mechanical:MountingHole
- added J7, J8: DIN41612_02x32_AB, Connector_DIN:DIN41612_B_2x32_Female_Vertical_THT, symbol Connector:DIN41612_02x32_AB
- J1: footprint Connector_PinHeader_2.54mm:PinHeader_1x04_P2.54mm_Vertical -> Connector_Molex:Molex_KK-396_A-41791-0004_1x04_P3.96mm_Vertical
Connections:
- net BA0: now also J7.a1 (Pin_a1), J8.a1 (Pin_a1)
- net BA1: now also J7.a2 (Pin_a2), J8.a2 (Pin_a2)
- net BA10: now also J7.a11 (Pin_a11), J8.a11 (Pin_a11)
- net BA11: now also J7.a12 (Pin_a12), J8.a12 (Pin_a12)
- net BA12: now also J7.a13 (Pin_a13), J8.a13 (Pin_a13)
- net BA13: now also J7.a14 (Pin_a14), J8.a14 (Pin_a14)
- net BA14: now also J7.a15 (Pin_a15), J8.a15 (Pin_a15)
- net BA15: now also J7.a16 (Pin_a16), J8.a16 (Pin_a16)
- net BA16: now also J7.a17 (Pin_a17), J8.a17 (Pin_a17)
- net BA17: now also J7.a18 (Pin_a18), J8.a18 (Pin_a18)
- net BA18: now also J7.a19 (Pin_a19), J8.a19 (Pin_a19)
- net BA19: now also J7.a20 (Pin_a20), J8.a20 (Pin_a20)
- net BA2: now also J7.a3 (Pin_a3), J8.a3 (Pin_a3)
- net BA3: now also J7.a4 (Pin_a4), J8.a4 (Pin_a4)
- net BA4: now also J7.a5 (Pin_a5), J8.a5 (Pin_a5)
- net BA5: now also J7.a6 (Pin_a6), J8.a6 (Pin_a6)
- net BA6: now also J7.a7 (Pin_a7), J8.a7 (Pin_a7)
- net BA7: now also J7.a8 (Pin_a8), J8.a8 (Pin_a8)
- net BA8: now also J7.a9 (Pin_a9), J8.a9 (Pin_a9)
- net BA9: now also J7.a10 (Pin_a10), J8.a10 (Pin_a10)
- net BCLK: now also J7.b23 (Pin_b23), J8.b23 (Pin_b23)
- net BD0: now also J7.a25 (Pin_a25), J8.a25 (Pin_a25)
- net BD1: now also J7.a26 (Pin_a26), J8.a26 (Pin_a26)
- net BD2: now also J7.a27 (Pin_a27), J8.a27 (Pin_a27)
- net BD3: now also J7.a28 (Pin_a28), J8.a28 (Pin_a28)
- net BD4: now also J7.a29 (Pin_a29), J8.a29 (Pin_a29)
- net BD5: now also J7.a30 (Pin_a30), J8.a30 (Pin_a30)
- net BD6: now also J7.a31 (Pin_a31), J8.a31 (Pin_a31)
- net BD7: now also J7.a32 (Pin_a32), J8.a32 (Pin_a32)
- net BIORQ: now also J7.a22 (Pin_a22), J8.a22 (Pin_a22)
- net BM1: now also J7.b22 (Pin_b22), J8.b22 (Pin_b22)
- net BMREQ: now also J7.a21 (Pin_a21), J8.a21 (Pin_a21)
- net BRD: now also J7.a23 (Pin_a23), J8.a23 (Pin_a23)
- net BWR: now also J7.a24 (Pin_a24), J8.a24 (Pin_a24)
- net GND: now also J7.b10 (Pin_b10), J7.b11 (Pin_b11), J7.b12 (Pin_b12), J7.b13 (Pin_b13), J7.b14 (Pin_b14), J7.b15 (Pin_b15), J7.b16 (Pin_b16), J7.b25 (Pin_b25), J7.b26 (Pin_b26), J7.b27 (Pin_b27), J7.b28 (Pin_b28), J7.b29 (Pin_b29), J7.b30 (Pin_b30), J7.b31 (Pin_b31), J7.b32 (Pin_b32), J7.b5 (Pin_b5), J7.b6 (Pin_b6), J7.b7 (Pin_b7), J7.b8 (Pin_b8), J7.b9 (Pin_b9), J8.b10 (Pin_b10), J8.b11 (Pin_b11), J8.b12 (Pin_b12), J8.b13 (Pin_b13), J8.b14 (Pin_b14), J8.b15 (Pin_b15), J8.b16 (Pin_b16), J8.b25 (Pin_b25), J8.b26 (Pin_b26), J8.b27 (Pin_b27), J8.b28 (Pin_b28), J8.b29 (Pin_b29), J8.b30 (Pin_b30), J8.b31 (Pin_b31), J8.b32 (Pin_b32), J8.b5 (Pin_b5), J8.b6 (Pin_b6), J8.b7 (Pin_b7), J8.b8 (Pin_b8), J8.b9 (Pin_b9)
- net VCC: now also J7.b1 (Pin_b1), J7.b2 (Pin_b2), J7.b3 (Pin_b3), J7.b4 (Pin_b4), J8.b1 (Pin_b1), J8.b2 (Pin_b2), J8.b3 (Pin_b3), J8.b4 (Pin_b4)
Other:
- moved on the sheet: C1, C10, C11, C12, C13, C14, C2, C3, C4, C5, C6, C7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

Commit message: add VR
Parts:
- added C15, C16: .01uF, Capacitor_THT:C_Disc_D5.0mm_W2.5mm_P2.50mm, symbol Device:C_Small
- added D4, D5: LED, LED_THT:LED_D3.0mm, symbol Device:LED
- added DS1: RC1602A, Connector_PinHeader_2.54mm:PinHeader_2x08_P2.54mm_Vertical, symbol Display_Character:RC1602A
- added R14, R15: 1k, Resistor_THT:R_Axial_DIN0207_L6.3mm_D2.5mm_P10.16mm_Horizontal, symbol Device:R_US
- added R16: 470, Resistor_THT:R_Axial_DIN0207_L6.3mm_D2.5mm_P10.16mm_Horizontal, symbol Device:R
- added RV1: 10k, Potentiometer_THT:Potentiometer_Bourns_3266W_Vertical, symbol Device:R_Potentiometer
- added U10: 74LS374, Package_DIP:DIP-20_W7.62mm, symbol 74xx:74LS374
- added U14: LM7805_TO220, Package_TO_SOT_THT:TO-220-3_Vertical, symbol Regulator_Linear:LM7805_TO220
- renumbered C12 to C10, C8 to C11, C11 to C12, C6 to C5, C7 to C6, C9 to C7, C5 to C8, C10 to C9, J7 to J3, J8 to J4, J3 to J5, J4 to J6, J5 to J7, J6 to J8, U2 to U1, U10 to U12, U12 to U13, U1 to U2, U8 to U6, U6 to U8
Connections:
- net D0: now also U10.13 (D4)
- net D1: now also U10.14 (D5)
- net D2: now also U10.17 (D6)
- net D3: now also U10.18 (D7)
- net D4: now also U10.3 (D0)
- net D5: now also U10.4 (D1)
- net D6: now also U10.7 (D2)
- net D7: now also U10.8 (D3)
- net GND: now also C15.2, C16.2, DS1.1 (VSS), DS1.10 (DB3), DS1.5 (R/W), DS1.7 (DB0), DS1.8 (DB1), DS1.9 (DB2), R16.2, RV1.3, U10.1 (OE), U10.10 (GND), U14.2 (GND)
- net VCC: now also C15.1, D4.2 (A), D5.2 (A), DS1.15 (A/VEE), DS1.2 (VDD), RV1.1, U10.20 (VCC), U14.3 (VO); no longer J1.1 (Pin_1), J1.2 (Pin_2)
- net nLCD: now reaches U6.9 (O3)
- new net: C16.1, J1.1 (Pin_1), J1.2 (Pin_2), U14.1 (VI)
- new net: D4.1 (K), R14.1
- new net: DS1.11 (DB4), U10.12 (O4)
- new net: DS1.12 (DB5), U10.15 (O5)
- new net: DS1.13 (DB6), U10.16 (O6)
- new net: DS1.14 (DB7), U10.19 (O7)
- new net: DS1.16 (K), R16.1
- new net: DS1.3 (VO), RV1.2
- new net: D5.1 (K), R15.1
- new net EN: DS1.6 (E), U10.5 (O1)
- new net LED0: R14.2, U10.6 (O2)
- new net LED1: R15.2, U10.9 (O3)
- new net RS: DS1.4 (RS), U10.2 (O0)
Other:
- moved on the sheet: J1, J8, U12, U7A

Commit message: tweaking placement
Connections:
- net GND: now also U1.1 (OEa), U1.19 (OEb)
Other:
- note added: ""HALT""
- note added: ""LED1""
- note added: ""LED2""
- note added: ""LED3""
- note added: "1602 LCD"
- note added: "Decode IO: 0000 - 00FF = on-board I/O 1000 - 10FF = off-board I/O 2000 - 20FF = 8255 3000 - 30FF = LCD / LEDs (Incompletely decoded)"
- note added: "POWER in 7-9VDC"
- note added: "Parallel / IDE"
- note added: "Synchronous Serial"
- note added: "UPCO Z180 Motherboard"
- note removed: "Decode IO: 0000 - 00FF = on-board I/O 1000 - 10FF = off-board I/O 2000 - 20FF = 8255 3000 - 30FF = spare (Incompletely decoded)"
- note removed: "POWER"
- moved on the sheet: C15, C16, J1, J8, U12, U14, U7A
